File: hardware/power.kicad_sch (KiCad schematic)
At the start: 1 part, among them U1 RK3562

Commit message: DDR4 schematic almost completed
Changed lines of the file:
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@@
 		(dnp no)
 		(property "Reference" "U1"
-			(at 274.13 93.98 0)
+			(at 280.162 94.742 0)
 			(effects
 				(font
@@
 		)
 		(property "Value" "RK3562"
-			(at 274.13 96.52 0)
+			(at 280.162 97.282 0)
 			(effects
 				(font
@@
 		)
 		(instances
-			(project "mini-server"
+			(project ""
+				(path "/17ecef2a-4000-49de-93ef-dcbfcfdaa69f/b0ac13bd-9621-484e-ac2a-625147906591"
+					(reference "U1")
+					(unit 5)
+				)
 				(path "/17ecef2a-4000-49de-93ef-dcbfcfdaa69f/e04d234d-f1f6-4b82-828e-fb6967cfc08b"
 					(reference "U1")
@@
 		(fields_autoplaced yes)
 		(property "Reference" "U1"
-			(at 59.69 31.75 0)
+			(at 59.69 80.01 0)
 			(effects
 				(font
@@
 		)
 		(property "Value" "RK3562"
-			(at 59.69 34.29 0)
+			(at 59.69 82.55 0)
 			(effects
 				(font
@@
 		)
 		(instances
-			(project "mini-server"
+			(project ""
+				(path "/17ecef2a-4000-49de-93ef-dcbfcfdaa69f/b0ac13bd-9621-484e-ac2a-625147906591"
+					(reference "U1")
+					(unit 6)
+				)
 				(path "/17ecef2a-4000-49de-93ef-dcbfcfdaa69f/e04d234d-f1f6-4b82-828e-fb6967cfc08b"
 					(reference "U1")
