File: hardware/HDMI.kicad_sch (KiCad schematic)
At the start: 1 part, among them J2 HDMI_A

Commit message: Routing and PCB
Parts:
- added C58: 100n, Capacitor_SMD:C_0201_0603Metric, symbol Device:C_Small
- added U3: TPD12S016PWR, easyeda2kicad:TSSOP-24_L7.8-W4.4-P0.65-LS6.4-BL, symbol easyeda2kicad:TPD12S016PWR
Connections:
- net HDMI_TX2P: now reaches J2.1 (D2+)
- net HDMI_TX2P: now also U3.23 (D2+)
- net HDMI_CLKP: now reaches J2.10 (CK+)
- net HDMI_CLKP: now also U3.16 (CLK+)
- net GND: now reaches J2.11 (CKS)
- net GND: now also J2.17 (GND), J2.2 (D2S), J2.5 (D1S), J2.8 (D0S), J2.SH, C58.2, U3.14 (GND), U3.19 (GND), U3.6 (GND)
- net HDMI_CLKN: now reaches J2.12 (CK-)
- net HDMI_CLKN: now also U3.15 (CLK-)
- net at J2.13 (CEC): now also U3.7 (CEC_B)
- net at J2.15 (SCL): now also U3.8 (SCL_B)
- net at J2.16 (SDA): now also U3.9 (SDA_B)
- net at J2.18 (+5V): now also C58.1, U3.13 (5V_OUT)
- net at J2.19 (HPD): now also U3.10 (HPD_B)
- net HDMI_TX2N: now reaches J2.3 (D2-)
- net HDMI_TX2N: now also U3.22 (D2-)
- net HDMI_TX1P: now reaches J2.4 (D1+)
- net HDMI_TX1P: now also U3.21 (D1+)
- net HDMI_TX1N: now reaches J2.6 (D1-)
- net HDMI_TX1N: now also U3.20 (D1-)
- net HDMI_TX0P: now reaches J2.7 (D0+)
- net HDMI_TX0P: now also U3.18 (D0+)
- net HDMI_TX0N: now reaches J2.9 (D0-)
- net HDMI_TX0N: now also U3.17 (D0-)
- new net +3V3: U3.12 (CT_HPD), U3.24 (VCCA), U3.5 (LS_OE)
- new net HDMI_CEC: U3.1 (CEC_A)
- new net HDMI_HPD: U3.4 (HPD_A)
- new net HDMI_SCL: U3.2 (SCL_A)
- new net HDMI_SDA: U3.3 (SDA_A)
- new net VSYS: U3.11 (VCC5V)
- no-connect marks 0 -> 1
Other:
- note added: "connect VCCA!"

Commit message: component Placement
Other:
- note removed: "connect VCCA!"
Changed lines of the file:
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@@
 	(generator_version "10.0")
 	(paper "A4")
-	(text "connect VCCA!"
-		(exclude_from_sim no)
-		(at 110.744 65.024 0)
-		(effects
-			(font
-				(size 1.27 1.27)
-			)
-		)
-	)
 	(junction
 		(at 138.43 104.14)
