File: hardware/mini-server.kicad_pcb (KiCad board)
At the start: 6 copper layers, 25 parts, among them U1 NT5CB256M16ER-FL, U2 RK3328

Commit message: stuff
Parts:
- added C20: 10u, Capacitor_SMD:C_0603_1608Metric, F.Cu at (58.5, 80.7)
- added C21: 100n, Capacitor_SMD:C_0201_0603Metric, B.Cu at (131.9, 94.5)
- added C22: 100n, Capacitor_SMD:C_0201_0603Metric, B.Cu at (131.2, 93.1)
- added C23: 100n, Capacitor_SMD:C_0201_0603Metric, B.Cu at (130.9, 94.2)
- added C24: 100n, Capacitor_SMD:C_0201_0603Metric, B.Cu at (128.2, 93.6)
- added C25: 100n, Capacitor_SMD:C_0201_0603Metric, B.Cu at (129.0, 93.8)
- added C26: 100n, Capacitor_SMD:C_0201_0603Metric, B.Cu at (128.5, 91.8)
- added C27: 100n, Capacitor_SMD:C_0201_0603Metric, B.Cu at (128.0, 92.3)
- added C28: 100n, Capacitor_SMD:C_0201_0603Metric, B.Cu at (126.6, 91.6)
- added C29: 100n, Capacitor_SMD:C_0201_0603Metric, B.Cu at (125.5, 95.8)
- added C30: 100n, Capacitor_SMD:C_0201_0603Metric, B.Cu at (127.2, 89.4)
- added C31: 100n, Capacitor_SMD:C_0201_0603Metric, B.Cu at (131.9, 93.1)
- added C32: 100n, Capacitor_SMD:C_0201_0603Metric, B.Cu at (130.0, 92.8)
- added C33: 100n, Capacitor_SMD:C_0201_0603Metric, B.Cu at (129.4, 92.4)
- added C34: 10u, Capacitor_SMD:C_0603_1608Metric, F.Cu at (58.5, 79.3)
- added C35: 100n, Capacitor_SMD:C_0201_0603Metric, F.Cu at (59.2, 78.2)
- added C36: 10u, Capacitor_SMD:C_0603_1608Metric, F.Cu at (63.4, 80.5)
- added C37: 100n, Capacitor_SMD:C_0201_0603Metric, F.Cu at (63.3, 82.4)
- added C38: 10u, Capacitor_SMD:C_0603_1608Metric, F.Cu at (57.9, 90.1)
- added C39: 10u, Capacitor_SMD:C_0603_1608Metric, F.Cu at (57.9, 91.6)
- added C40: 100n, Capacitor_SMD:C_0201_0603Metric, F.Cu at (58.7, 89.0)
- added C41: 10u, Capacitor_SMD:C_0603_1608Metric, F.Cu at (63.6, 92.3)
- added C42: 100n, Capacitor_SMD:C_0201_0603Metric, F.Cu at (62.8, 93.4)
- added C43: 10u, Capacitor_SMD:C_0603_1608Metric, F.Cu at (84.0, 80.8)
- added C44: 10u, Capacitor_SMD:C_0603_1608Metric, F.Cu at (84.0, 83.3)
- added C45: 10u, Capacitor_SMD:C_0603_1608Metric, F.Cu at (88.0, 75.8)
- added C46: 10u, Capacitor_SMD:C_0603_1608Metric, F.Cu at (88.0, 78.3)
- added C47: 100n, Capacitor_SMD:C_0201_0603Metric, F.Cu at (79.2, 92.5)
- added C48: 100n, Capacitor_SMD:C_0201_0603Metric, F.Cu at (79.2, 94.2)
- added C49: 10u, Capacitor_SMD:C_0603_1608Metric, F.Cu at (88.0, 80.8)
- added C50: 10u, Capacitor_SMD:C_0603_1608Metric, F.Cu at (88.0, 83.3)
- added C51: 100n, Capacitor_SMD:C_0201_0603Metric, F.Cu at (81.7, 85.5)
- added C52: 100n, Capacitor_SMD:C_0201_0603Metric, F.Cu at (81.7, 87.2)
- added J2: HDMI_A, Connector_Video:HDMI_A_Molex_208658-1001_Horizontal, F.Cu at (97.9, 80.5)
- added J3: Micro_SD_Card, Connector_Card:microSD_HC_Molex_104031-0811, F.Cu at (99.6, 101.8)
- added L1: 2.2u, Inductor_SMD:L_1008_2520Metric, F.Cu at (61.3, 80.7)
- added L2: 2.2u, Inductor_SMD:L_1008_2520Metric, F.Cu at (60.8, 91.8)
- added L3: 2.2u, Inductor_SMD:L_1008_2520Metric, F.Cu at (75.5, 80.8)
- added L4: 2.2u, Inductor_SMD:L_1008_2520Metric, F.Cu at (75.5, 84.6)
- added Q1: 2N7002, Package_TO_SOT_SMD:SOT-23, F.Cu at (57.7, 76.3)
- added R10: R, Resistor_SMD:R_0201_0603Metric, F.Cu at (84.1, 89.0)
- added R11: R, Resistor_SMD:R_0201_0603Metric, F.Cu at (84.1, 90.7)
- added R12: R, Resistor_SMD:R_0201_0603Metric, F.Cu at (59.3, 77.2)
- added R4: R, Resistor_SMD:R_0201_0603Metric, B.Cu at (61.1, 78.3)
- added R5: R, Resistor_SMD:R_0201_0603Metric, B.Cu at (60.4, 76.9)
- added R6: R, Resistor_SMD:R_0201_0603Metric, B.Cu at (60.7, 89.1)
- added R7: R, Resistor_SMD:R_0201_0603Metric, B.Cu at (60.6, 87.9)
- added R8: R, Resistor_SMD:R_0201_0603Metric, F.Cu at (84.1, 85.5)
- added R9: R, Resistor_SMD:R_0201_0603Metric, F.Cu at (84.1, 87.2)
- added RJ1: HR911130A, easyeda2kicad:RJ45-TH_HR911130A, F.Cu at (167.5, 77.9)
- added U4: RTL8211F-CG, Package_DFN_QFN:VQFN-40-1EP_5x5mm_P0.4mm_EP3.7x3.7mm, F.Cu at (77.7, 101.5)
- added U6: TPS563252DRLR, easyeda2kicad:SOT-563-6_L1.6-W1.2-P0.50-LS1.6-BL, F.Cu at (61.1, 77.6)
- added U7: TPS563252DRLR, easyeda2kicad:SOT-563-6_L1.6-W1.2-P0.50-LS1.6-BL, F.Cu at (60.8, 88.4)
- added U8: TPS563252DRLR, easyeda2kicad:SOT-563-6_L1.6-W1.2-P0.50-LS1.6-BL, F.Cu at (85.7, 72.9)
- added U9: TPS563252DRLR, easyeda2kicad:SOT-563-6_L1.6-W1.2-P0.50-LS1.6-BL, F.Cu at (88.8, 72.9)
Connections:
- U2 pad H5: unconnected-(U2B-PLL_AVDD_1V8-PadH5) -> +1V8
- U2 pad H7: unconnected-(U2B-PLL_DVDD_1V0-PadH7) -> +1V0
- U2 pad J5: unconnected-(U2B-USB30_AVDD_1V8-PadJ5) -> +1V8
- U2 pad J6: unconnected-(U2B-USB30_AVDD_3V3-PadJ6) -> +3V3
- U2 pad J7: unconnected-(U2B-USB30_DVDD_1V0-PadJ7) -> +1V0
- U2 pad K6: unconnected-(U2B-VCCIO_PMU-PadK6) -> +3V3
- U2 pad M16: unconnected-(U2B-SARADC_AVDD_1V8-PadM16) -> +1V8
- U2 pad M6: unconnected-(U2B-HDMI_AVDD_1V0-PadM6) -> +1V0
- U2 pad N10: Net-(U2B-VDD_LOGIC_1) -> +1V0
- U2 pad N11: Net-(U2B-VDD_LOGIC_1) -> +1V0
- U2 pad N5: unconnected-(U2B-CODEC_AVDD_1V8-PadN5) -> +1V8
- U2 pad N6: unconnected-(U2B-VDAC_AVDD_1V8-PadN6) -> +1V8
- U2 pad N9: Net-(U2B-VDD_LOGIC_1) -> +1V0
- U2 pad P10: Net-(U2B-VDD_LOGIC_1) -> +1V0
- U2 pad P11: Net-(U2B-VDD_LOGIC_1) -> +1V0
- U2 pad P13: Net-(U2B-VDD_CORE_1) -> +1V0
- U2 pad P14: Net-(U2B-VDD_CORE_1) -> +1V0
- U2 pad P6: unconnected-(U2B-HDMI_AVDD_1V8-PadP6) -> +1V8
- U2 pad P9: Net-(U2B-VDD_LOGIC_1) -> +1V0
- U2 pad R10: Net-(U2B-VDD_LOGIC_1) -> +1V0
- U2 pad R11: Net-(U2B-VDD_LOGIC_1) -> +1V0
- U2 pad R13: Net-(U2B-VDD_CORE_1) -> +1V0
- U2 pad R14: Net-(U2B-VDD_CORE_1) -> +1V0
- U2 pad R9: Net-(U2B-VDD_LOGIC_1) -> +1V0
- U2 pad T13: Net-(U2B-VDD_CORE_1) -> +1V0
- U2 pad T14: Net-(U2B-VDD_CORE_1) -> +1V0
- U2 pad T15: Net-(U2B-VDD_CORE_1) -> +1V0
- U2 pad T5: unconnected-(U2B-USB20_AVDD_3V3-PadT5) -> +3V3
- U2 pad T7: unconnected-(U2B-VCCIO1-PadT7) -> +3V3
- U2 pad U5: unconnected-(U2B-USB20_AVDD_1V8-PadU5) -> +1V8
- U2 pad U6: unconnected-(U2B-FEPHY_AVDD_1V8-PadU6) -> +1V8
- U2 pad V5: unconnected-(U2B-USB20_DVDD_1V0-PadV5) -> +1V0
- U2 pad V6: unconnected-(U2B-FEPHY_AVDD_1V0-PadV6) -> +1V0
Routing:
- net +1V0: track 0.00 -> 14.2 mm, vias 0 -> 19
- net Net-(U2B-VDD_LOGIC_1): track 7.40 -> 0.00 mm
- net Net-(U2B-VDD_CORE_1): track 5.25 -> 0.00 mm
- net +1V8: track 0.00 -> 3.02 mm, vias 0 -> 2
- net VSYS: track 0.00 -> 1.61 mm
- net Net-(U7-FB): track 0.00 -> 1.58 mm, vias 0 -> 1
- net +3V3: track 0.00 -> 0.70 mm, vias 0 -> 3
- net Net-(U6-SW): track 0.00 -> 0.67 mm, vias 0 -> 1
- net Net-(U6-FB): track 0.00 -> 0.38 mm, vias 0 -> 1
- net Net-(U7-SW): track 0.00 -> 0.10 mm, vias 0 -> 1
- net unconnected-(U2H-CODEC_VCM-PadT4): track 0.00 -> 0.06 mm, vias 0 -> 1
- net unconnected-(U2G-USB20_VBUS-PadT6): vias 0 -> 1
- net GND: vias 30 -> 38
- net +1V5: vias 22 -> 31
- added copper zone on F.Cu, net +1V0
- added copper zone on F.Cu, net +1V5
- added copper zone on F.Cu, net Net-(U6-SW)
- added copper zone on F.Cu, net Net-(U7-SW)

Commit message: stuff
Parts:
- removed RJ1: HR911130A, easyeda2kicad:RJ45-TH_HR911130A
- removed U4: RTL8211F-CG, Package_DFN_QFN:VQFN-40-1EP_5x5mm_P0.4mm_EP3.7x3.7mm
- added C53: 100n, Capacitor_SMD:C_0201_0603Metric, F.Cu at (131.1, 100.3)
- added C54: 100n, Capacitor_SMD:C_0201_0603Metric, F.Cu at (131.1, 102.0)
- added C55: 100n, Capacitor_SMD:C_0201_0603Metric, F.Cu at (102.1, 68.7)
- added J1: RJ45_Hanrun_HR911105A_Horizontal, Connector_RJ:RJ45_Hanrun_HR911105A_Horizontal, F.Cu at (115.4, 104.5)
- R10, R11, R8, R9: moved to B.Cu
- U1: footprint Package_BGA:FBGA-96_8x13mm_Layout9x16_P0.8mm -> easyeda2kicad:TFBGA-96_L13.0-W8.0-R16-C6-P0.80-TL
- moved C45 42.2 mm to (57.4, 104.8), turned to 180 degrees
- moved U8 39.6 mm to (60.3, 103.3)
- moved J3 38.4 mm to (137.3, 109.2)
- moved C43 36.8 mm to (57.4, 106.3), turned to 180 degrees
- moved C49 36.3 mm to (63.1, 107.1)
- moved R8 30.3 mm to (60.3, 104.2), turned to 90 degrees
- moved L3 30.0 mm to (60.3, 106.6), turned to -90 degrees
- moved C51 29.9 mm to (62.3, 108.2)
- moved U9 29.7 mm to (91.5, 102.5)
- moved R9 29.2 mm to (59.4, 102.7), turned to 90 degrees
- moved L4 26.7 mm to (91.6, 105.9), turned to -90 degrees
- moved C46 26.0 mm to (88.7, 104.3), turned to 180 degrees
- moved C50 23.9 mm to (94.4, 106.4)
- moved C47 23.9 mm to (58.2, 103.7), turned to 180 degrees
- moved C52 23.5 mm to (93.6, 107.5)
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Connections:
- C18 pad 2: Net-(U1-VREFCA) -> Net-(U1-A0)
- C19 pad 1: Net-(U1-VREFCA) -> Net-(U1-A0)
- J3 pad 1: unconnected-(J3-DAT2-Pad1) -> /Storage/SD_DAT2
- J3 pad 2: unconnected-(J3-DAT3/CD-Pad2) -> /Storage/SD_DAT3
- J3 pad 3: unconnected-(J3-CMD-Pad3) -> /Storage/SD_CMD
- J3 pad 4: unconnected-(J3-VDD-Pad4) -> +3V3
- J3 pad 5: unconnected-(J3-CLK-Pad5) -> /Storage/SD_CLK
- J3 pad 6: unconnected-(J3-VSS-Pad6) -> GND
- J3 pad 7: unconnected-(J3-DAT0-Pad7) -> /Storage/SD_DAT0
- J3 pad 8: unconnected-(J3-DAT1-Pad8) -> /Storage/SD_DAT1
- R1 pad 1: Net-(U1-ZQ) -> unconnected-(R1-Pad1)
- R2 pad 2: Net-(U1-VREFCA) -> Net-(U1-A0)
- R3 pad 1: Net-(U1-VREFCA) -> Net-(U1-A0)
- U1 pad A2: /DDR3/DQU4 -> +1V5
- U1 pad A3: /DDR3/DQU7 -> +1V5
- U1 pad A7: /DDR3/DQU0 -> +1V5
- U1 pad A9: GND -> +1V5
- U1 pad B1: GND -> +1V5
- U1 pad B3: GND -> +1V5
- U1 pad B7: /DDR3/DQSUN -> unconnected-(U1-~{DQSU}-PadB7)
- U1 pad B8: /DDR3/DQU2 -> /DDR3/DQU5
- U1 pad B9: GND -> /DDR3/DQU1
- U1 pad C1: +1V5 -> /DDR3/DQU6
- U1 pad C3: /DDR3/DQU1 -> /DDR3/DQU0
- U1 pad C7: /DDR3/DQSUP -> /DDR3/DQU4
- U1 pad C8: /DDR3/DQU6 -> /DDR3/DQU2
- U1 pad C9: +1V5 -> /DDR3/DQU7
- U1 pad D1: GND -> /DDR3/DQL6
- U1 pad D2: +1V5 -> /DDR3/DQL3
- U1 pad D3: /DDR3/DMU -> /DDR3/DQL4
- U1 pad D7: /DDR3/DQU5 -> /DDR3/DQL7
- U1 pad D8: GND -> /DDR3/DQL5
- U1 pad D9: +1V5 -> /DDR3/DQL1
- U1 pad E1: GND -> /DDR3/DQL0
- U1 pad E2: GND -> /DDR3/DQL2
- U1 pad E3: /DDR3/DQL6 -> unconnected-(U1-DQL0-PadE3)
- U1 pad E7: /DDR3/DML -> unconnected-(U1-DML-PadE7)
- U1 pad E8: GND -> unconnected-(U1-VSSQ-PadE8)
- U1 pad E9: +1V5 -> unconnected-(U1-VDDQ-PadE9)
- U1 pad F1: +1V5 -> unconnected-(U1-VDDQ-PadF1)
- U1 pad F2: /DDR3/DQL4 -> unconnected-(U1-DQL2-PadF2)
- U1 pad F3: /DDR3/DQSLP -> unconnected-(U1-DQSL-PadF3)
- U1 pad F7: /DDR3/DQL3 -> unconnected-(U1-DQL1-PadF7)
- U1 pad F8: /DDR3/DQL7 -> unconnected-(U1-DQL3-PadF8)
- U1 pad F9: GND -> unconnected-(U1-VSSQ-PadF9)
- U1 pad G1: GND -> unconnected-(U1-VSSQ-PadG1)
- U1 pad G2: /DDR3/DQL0 -> unconnected-(U1-DQL6-PadG2)
- U1 pad G3: /DDR3/DQSLN -> unconnected-(U1-~{DQSL}-PadG3)
- U1 pad G7: +1V5 -> unconnected-(U1-VDD-PadG7)
- U1 pad G8: GND -> unconnected-(U1-VSS-PadG8)
- U1 pad G9: GND -> unconnected-(U1-VSSQ-PadG9)
- U1 pad H1: Net-(U1-VREFCA) -> unconnected-(U1-VREFDQ-PadH1)
- U1 pad H2: +1V5 -> unconnected-(U1-VDDQ-PadH2)
- U1 pad H3: /DDR3/DQL5 -> unconnected-(U1-DQL4-PadH3)
- U1 pad H7: /DDR3/DQL2 -> unconnected-(U1-DQL7-PadH7)
- U1 pad H8: /DDR3/DQL1 -> unconnected-(U1-DQL5-PadH8)
- U1 pad H9: +1V5 -> unconnected-(U1-VDDQ-PadH9)
- U1 pad J1: GND -> +1V5
- U1 pad J2: GND -> +1V5
- U1 pad J3: /DDR3/RASn -> +1V5
- U1 pad J7: /DDR3/CKP -> +1V5
- U1 pad J8: GND -> +1V5
- U1 pad J9: GND -> +1V5
- U1 pad K1: /DDR3/ODT -> +1V5
- U1 pad K3: /DDR3/CASn -> +1V5
- U1 pad K7: /DDR3/CKN -> unconnected-(U1-~{CK}-PadK7)
- U1 pad K8: +1V5 -> /DDR3/A0
- U1 pad K9: /DDR3/CKE -> /DDR3/A1
- U1 pad L1: GND -> /DDR3/A2
- U1 pad L2: /DDR3/CSn -> /DDR3/A3
- U1 pad L3: /DDR3/WEn -> /DDR3/A4
- U1 pad L7: /DDR3/A10 -> /DDR3/A5
- U1 pad L8: Net-(U1-ZQ) -> /DDR3/A6
- U1 pad L9: GND -> /DDR3/A7
- U1 pad M1: GND -> /DDR3/A8
- U1 pad M2: /DDR3/BA0 -> /DDR3/A9
- U1 pad M3: /DDR3/BA2 -> /DDR3/A10
- U1 pad M7: GND -> /DDR3/A11
- U1 pad M8: Net-(U1-VREFCA) -> /DDR3/A12
- U1 pad M9: GND -> /DDR3/A13
- U1 pad N1: +1V5 -> /DDR3/A14
- U1 pad N2: /DDR3/A3 -> unconnected-(U1-A3-PadN2)
- U1 pad N3: /DDR3/A0 -> Net-(U1-A0)
- U1 pad N7: /DDR3/A12 -> unconnected-(U1-A12/~{BC}-PadN7)
- U1 pad N8: /DDR3/BA1 -> unconnected-(U1-BA1-PadN8)
- U1 pad N9: +1V5 -> unconnected-(U1-VDD-PadN9)
- U1 pad P1: GND -> unconnected-(U1-VSS-PadP1)
- U1 pad P2: /DDR3/A5 -> unconnected-(U1-A5-PadP2)
- U1 pad P3: /DDR3/A2 -> unconnected-(U1-A2-PadP3)
- U1 pad P7: /DDR3/A1 -> unconnected-(U1-A1-PadP7)
- U1 pad P8: /DDR3/A4 -> unconnected-(U1-A4-PadP8)
- U1 pad P9: GND -> unconnected-(U1-VSS-PadP9)
- U1 pad R1: +1V5 -> unconnected-(U1-VDD-PadR1)
- U1 pad R2: /DDR3/A7 -> unconnected-(U1-A7-PadR2)
- U1 pad R3: /DDR3/A9 -> unconnected-(U1-A9-PadR3)
- U1 pad R7: /DDR3/A11 -> unconnected-(U1-A11-PadR7)
- U1 pad R8: /DDR3/A6 -> unconnected-(U1-A6-PadR8)
- U1 pad R9: +1V5 -> unconnected-(U1-VDD-PadR9)
- U1 pad T1: GND -> unconnected-(U1-VSS-PadT1)
- U1 pad T2: /DDR3/RSTn -> unconnected-(U1-~{RESET}-PadT2)
- U1 pad T3: /DDR3/A13 -> unconnected-(U1-A13-PadT3)
- U1 pad T7: /DDR3/A14 -> unconnected-(U1-A14-PadT7)
- U1 pad T8: /DDR3/A8 -> unconnected-(U1-A8-PadT8)
- U1 pad T9: GND -> unconnected-(U1-VSS-PadT9)
- U2 pad AA13: unconnected-(U2F-GPIO1_A3/SDMMC0_D3/JTAG_TMS-PadAA13) -> /Storage/SD_DAT3
- U2 pad AA8: unconnected-(U2E-FEPHY_RXN-PadAA8) -> /Ethernet/PHY_RXN
- U2 pad AA9: unconnected-(U2E-FEPHY_TXN-PadAA9) -> /Ethernet/PHY_TXN
- U2 pad P17: unconnected-(U2H-GPIO2_D0/I2C0_SCL/FEPHY_LED_LINK_M1-PadP17) -> /Ethernet/PHY_LINK_LED
- U2 pad R17: unconnected-(U2H-GPIO2_D1/I2C0_SDA/FEPHY_LED_DATA_M1-PadR17) -> /Ethernet/PHY_DATA_LED
- U2 pad U10: unconnected-(U2F-GPIO1_A0/SDMMC0_D0/UART2_TX_M0-PadU10) -> /Storage/SD_DAT0
- U2 pad V10: unconnected-(U2F-GPIO1_A5/SDMMC0_DETN-PadV10) -> /main/SD_DETN
- U2 pad V7: unconnected-(U2E-FEPHY_EXTRES-PadV7) -> Net-(U2E-FEPHY_EXTRES)
- U2 pad W11: unconnected-(U2F-GPIO1_A1/SDMMC0_D1/UART2_RX_M0-PadW11) -> /Storage/SD_DAT1
- U2 pad W12: unconnected-(U2F-GPIO1_A6/SDMMC0_CLK/TEST_CLK0-PadW12) -> /Storage/SD_CLK
- U2 pad W13: unconnected-(U2F-GPIO1_A2/SDMMC0_D2/JTAG_TCK-PadW13) -> /Storage/SD_DAT2
- U2 pad Y13: unconnected-(U2F-GPIO1_A4/SDMMC0_CMD-PadY13) -> /Storage/SD_CMD
- U2 pad Y8: unconnected-(U2E-FEPHY_RXP-PadY8) -> /Ethernet/PHY_RXP
- U2 pad Y9: unconnected-(U2E-FEPHY_TXP-PadY9) -> /Ethernet/PHY_TXP
Routing:
- net (no net): track 0.00 -> 18.4 mm, vias 0 -> 3
- net Net-(U1-VREFCA): track 18.2 -> 0.00 mm, vias 2 -> 0
- net GND: track 157.9 -> 152.2 mm, vias 38 -> 33
- net unconnected-(U1-VSS-PadP1): track 0.00 -> 3.24 mm, vias 0 -> 1
- net Net-(U9-FB): track 0.00 -> 2.07 mm, vias 0 -> 1
- net Net-(U8-FB): track 0.00 -> 1.81 mm, vias 0 -> 1
- net unconnected-(U1-VSS-PadT1): track 0.00 -> 1.58 mm, vias 0 -> 1
- net Net-(U6-FB): track 0.38 -> 1.44 mm
- net Net-(U9-SW): track 0.00 -> 0.81 mm, vias 0 -> 1
- net Net-(U8-SW): track 0.00 -> 0.72 mm, vias 0 -> 1
- net /DDR3/A2: track 26.2 -> 26.8 mm, vias 2 -> 3
- net unconnected-(U1-VSSQ-PadG1): track 0.00 -> 0.27 mm, vias 0 -> 1
- net Net-(U1-ZQ): track 0.18 -> 0.00 mm, vias 1 -> 0
- net unconnected-(U1-VSS-PadP9): track 0.00 -> 0.02 mm, vias 0 -> 1
- net +1V8: vias 2 -> 10
- added copper zone on F.Cu, net +1V8
- added copper zone on F.Cu, net +3V3
- added copper zone on F.Cu, net Net-(U8-SW)
- added copper zone on F.Cu, net Net-(U9-SW)

Commit message: Routing and PCB
Parts:
- added C56: 10u, Capacitor_SMD:C_0603_1608Metric, F.Cu at (103.5, 72.4)
- added C57: 10u, Capacitor_SMD:C_0603_1608Metric, F.Cu at (103.5, 74.9)
- added C58: 100n, Capacitor_SMD:C_0201_0603Metric, B.Cu at (95.7, 84.4)
- added C59: 10u, Capacitor_SMD:C_0603_1608Metric, B.Cu at (125.1, 92.0)
- added J5: AudioJack4, Connector_Audio:Jack_3.5mm_KoreanHropartsElec_PJ-320D-4A_Horizontal, F.Cu at (90.3, 73.3)
- added J6: USB_C_Receptacle, Connector_USB:USB_C_Receptacle_Molex_105450-0101, F.Cu at (106.4, 61.5)
- added J7: USB_C_Receptacle, Connector_USB:USB_C_Receptacle_Molex_105450-0101, F.Cu at (173.3, 92.2)
- added J8: USB_C_Receptacle, Connector_USB:USB_C_Receptacle_Molex_105450-0101, F.Cu at (173.3, 102.7)
- added U3: TPD12S016PWR, easyeda2kicad:TSSOP-24_L7.8-W4.4-P0.65-LS6.4-BL, F.Cu at (105.0, 90.1)
- moved C55 51.2 mm to (141.0, 102.0)
- moved C44 34.6 mm to (56.8, 119.0)
- moved C48 34.6 mm to (57.6, 116.4)
- moved L4 34.6 mm to (59.6, 119.1)
- moved R10 34.6 mm to (59.6, 116.8)
- moved R11 34.6 mm to (58.6, 115.1)
- moved C46 34.6 mm to (56.8, 117.5)
- moved C50 34.6 mm to (62.4, 119.6)
- moved C52 34.6 mm to (61.7, 120.7)
- moved U9 34.6 mm to (59.6, 115.7)
- moved J2 14.6 mm to (89.8, 88.8), turned to 180 degrees
- moved J3 7.79 mm to (144.4, 112.4)
- moved J1 7.69 mm to (120.0, 110.6)
Connections:
- net /Storage/SD_DAT0 renamed /Storage/SD_D0
- net /Storage/SD_DAT1 renamed /Storage/SD_D1
- net /Storage/SD_DAT2 renamed /Storage/SD_D2
- net /Storage/SD_DAT3 renamed /Storage/SD_D3
- C18 pad 2: Net-(U1-A0) -> Net-(U1-VREFCA)
- C19 pad 1: Net-(U1-A0) -> Net-(U1-VREFCA)
- J2 pad 1: unconnected-(J2-D2+-Pad1) -> /HDMI/HDMI_TX2P
- J2 pad 10: unconnected-(J2-CK+-Pad10) -> /HDMI/HDMI_CLKP
- J2 pad 11: unconnected-(J2-CKS-Pad11) -> GND
- J2 pad 12: unconnected-(J2-CK--Pad12) -> /HDMI/HDMI_CLKN
- J2 pad 13: unconnected-(J2-CEC-Pad13) -> Net-(J2-CEC)
- J2 pad 15: unconnected-(J2-SCL-Pad15) -> Net-(J2-SCL)
- J2 pad 16: unconnected-(J2-SDA-Pad16) -> Net-(J2-SDA)
- J2 pad 17: unconnected-(J2-GND-Pad17) -> GND
- J2 pad 18: unconnected-(J2-+5V-Pad18) -> Net-(J2-+5V)
- J2 pad 19: unconnected-(J2-HPD-Pad19) -> Net-(J2-HPD)
- J2 pad 2: unconnected-(J2-D2S-Pad2) -> GND
- J2 pad 3: unconnected-(J2-D2--Pad3) -> /HDMI/HDMI_TX2N
- J2 pad 4: unconnected-(J2-D1+-Pad4) -> /HDMI/HDMI_TX1P
- J2 pad 5: unconnected-(J2-D1S-Pad5) -> GND
- J2 pad 6: unconnected-(J2-D1--Pad6) -> /HDMI/HDMI_TX1N
- J2 pad 7: unconnected-(J2-D0+-Pad7) -> /HDMI/HDMI_TX0P
- J2 pad 8: unconnected-(J2-D0S-Pad8) -> GND
- J2 pad 9: unconnected-(J2-D0--Pad9) -> /HDMI/HDMI_TX0N
- J2 pad SH: unconnected-(J2-PadSH) -> GND
- R1 pad 1: unconnected-(R1-Pad1) -> Net-(U1-ZQ)
- R2 pad 2: Net-(U1-A0) -> Net-(U1-VREFCA)
- R3 pad 1: Net-(U1-A0) -> Net-(U1-VREFCA)
- U1 pad A2: +1V5 -> /DDR3/DQU4
- U1 pad A3: +1V5 -> /DDR3/DQU7
- U1 pad A7: +1V5 -> /DDR3/DQU0
- U1 pad A9: +1V5 -> GND
- U1 pad B1: +1V5 -> GND
- U1 pad B3: +1V5 -> GND
- U1 pad B7: unconnected-(U1-~{DQSU}-PadB7) -> /DDR3/DQSUN
- U1 pad B8: /DDR3/DQU5 -> /DDR3/DQU2
- U1 pad B9: /DDR3/DQU1 -> GND
- U1 pad C1: /DDR3/DQU6 -> +1V5
- U1 pad C3: /DDR3/DQU0 -> /DDR3/DQU1
- U1 pad C7: /DDR3/DQU4 -> /DDR3/DQSUP
- U1 pad C8: /DDR3/DQU2 -> /DDR3/DQU6
- U1 pad C9: /DDR3/DQU7 -> +1V5
- U1 pad D1: /DDR3/DQL6 -> GND
- U1 pad D2: /DDR3/DQL3 -> +1V5
- U1 pad D3: /DDR3/DQL4 -> /DDR3/DMU
- U1 pad D7: /DDR3/DQL7 -> /DDR3/DQU5
- U1 pad D8: /DDR3/DQL5 -> GND
- U1 pad D9: /DDR3/DQL1 -> +1V5
- U1 pad E1: /DDR3/DQL0 -> GND
- U1 pad E2: /DDR3/DQL2 -> GND
- U1 pad E3: unconnected-(U1-DQL0-PadE3) -> /DDR3/DQL6
- U1 pad E7: unconnected-(U1-DML-PadE7) -> /DDR3/DML
- U1 pad E8: unconnected-(U1-VSSQ-PadE8) -> GND
- U1 pad E9: unconnected-(U1-VDDQ-PadE9) -> +1V5
- U1 pad F1: unconnected-(U1-VDDQ-PadF1) -> +1V5
- U1 pad F2: unconnected-(U1-DQL2-PadF2) -> /DDR3/DQL4
- U1 pad F3: unconnected-(U1-DQSL-PadF3) -> /DDR3/DQSLP
- U1 pad F7: unconnected-(U1-DQL1-PadF7) -> /DDR3/DQL3
- U1 pad F8: unconnected-(U1-DQL3-PadF8) -> /DDR3/DQL7
- U1 pad F9: unconnected-(U1-VSSQ-PadF9) -> GND
- U1 pad G1: unconnected-(U1-VSSQ-PadG1) -> GND
- U1 pad G2: unconnected-(U1-DQL6-PadG2) -> /DDR3/DQL0
- U1 pad G3: unconnected-(U1-~{DQSL}-PadG3) -> /DDR3/DQSLN
- U1 pad G7: unconnected-(U1-VDD-PadG7) -> +1V5
- U1 pad G8: unconnected-(U1-VSS-PadG8) -> GND
- U1 pad G9: unconnected-(U1-VSSQ-PadG9) -> GND
- U1 pad H1: unconnected-(U1-VREFDQ-PadH1) -> Net-(U1-VREFCA)
- U1 pad H2: unconnected-(U1-VDDQ-PadH2) -> +1V5
- U1 pad H3: unconnected-(U1-DQL4-PadH3) -> /DDR3/DQL5
- U1 pad H7: unconnected-(U1-DQL7-PadH7) -> /DDR3/DQL2
- U1 pad H8: unconnected-(U1-DQL5-PadH8) -> /DDR3/DQL1
- U1 pad H9: unconnected-(U1-VDDQ-PadH9) -> +1V5
- U1 pad J1: +1V5 -> GND
- U1 pad J2: +1V5 -> GND
- U1 pad J3: +1V5 -> /DDR3/RASn
- U1 pad J7: +1V5 -> /DDR3/CKP
- U1 pad J8: +1V5 -> GND
- U1 pad J9: +1V5 -> GND
- U1 pad K1: +1V5 -> /DDR3/ODT
- U1 pad K3: +1V5 -> /DDR3/CASn
- U1 pad K7: unconnected-(U1-~{CK}-PadK7) -> /DDR3/CKN
- U1 pad K8: /DDR3/A0 -> +1V5
- U1 pad K9: /DDR3/A1 -> /DDR3/CKE
- U1 pad L1: /DDR3/A2 -> GND
- U1 pad L2: /DDR3/A3 -> /DDR3/CSn
- U1 pad L3: /DDR3/A4 -> /DDR3/WEn
- U1 pad L7: /DDR3/A5 -> /DDR3/A10
- U1 pad L8: /DDR3/A6 -> Net-(U1-ZQ)
- U1 pad L9: /DDR3/A7 -> GND
- U1 pad M1: /DDR3/A8 -> GND
- U1 pad M2: /DDR3/A9 -> /DDR3/BA0
- U1 pad M3: /DDR3/A10 -> /DDR3/BA2
- U1 pad M7: /DDR3/A11 -> GND
- U1 pad M8: /DDR3/A12 -> Net-(U1-VREFCA)
- U1 pad M9: /DDR3/A13 -> GND
- U1 pad N1: /DDR3/A14 -> +1V5
- U1 pad N2: unconnected-(U1-A3-PadN2) -> /DDR3/A3
- U1 pad N3: Net-(U1-A0) -> /DDR3/A0
- U1 pad N7: unconnected-(U1-A12/~{BC}-PadN7) -> /DDR3/A12
- U1 pad N8: unconnected-(U1-BA1-PadN8) -> /DDR3/BA1
- U1 pad N9: unconnected-(U1-VDD-PadN9) -> +1V5
- U1 pad P1: unconnected-(U1-VSS-PadP1) -> GND
- U1 pad P2: unconnected-(U1-A5-PadP2) -> /DDR3/A5
- U1 pad P3: unconnected-(U1-A2-PadP3) -> /DDR3/A2
- U1 pad P7: unconnected-(U1-A1-PadP7) -> /DDR3/A1
- U1 pad P8: unconnected-(U1-A4-PadP8) -> /DDR3/A4
- U1 pad P9: unconnected-(U1-VSS-PadP9) -> GND
- U1 pad R1: unconnected-(U1-VDD-PadR1) -> +1V5
- U1 pad R2: unconnected-(U1-A7-PadR2) -> /DDR3/A7
- U1 pad R3: unconnected-(U1-A9-PadR3) -> /DDR3/A9
- U1 pad R7: unconnected-(U1-A11-PadR7) -> /DDR3/A11
- U1 pad R8: unconnected-(U1-A6-PadR8) -> /DDR3/A6
- U1 pad R9: unconnected-(U1-VDD-PadR9) -> +1V5
- U1 pad T1: unconnected-(U1-VSS-PadT1) -> GND
- U1 pad T2: unconnected-(U1-~{RESET}-PadT2) -> /DDR3/RSTn
- U1 pad T3: unconnected-(U1-A13-PadT3) -> /DDR3/A13
- U1 pad T7: unconnected-(U1-A14-PadT7) -> /DDR3/A14
- U1 pad T8: unconnected-(U1-A8-PadT8) -> /DDR3/A8
- U1 pad T9: unconnected-(U1-VSS-PadT9) -> GND
- U2 pad AA2: unconnected-(U2D-HDMI_TX0P-PadAA2) -> /HDMI/HDMI_TX0P
- U2 pad AA4: unconnected-(U2D-HDMI_TX2N-PadAA4) -> /HDMI/HDMI_TX2N
- U2 pad AA6: unconnected-(U2G-USB0_DP-PadAA6) -> /USB/USB2_0_DP
- U2 pad AA7: unconnected-(U2G-USB1_DP-PadAA7) -> /USB/USB2_1_DP
- U2 pad G5: unconnected-(U2G-USB30_EXTR-PadG5) -> Net-(U2G-USB30_EXTR)
- U2 pad H2: unconnected-(U2G-USB30_TXN-PadH2) -> /USB/USB3_TXN
- U2 pad H3: unconnected-(U2G-USB30_TXP-PadH3) -> /USB/USB3_TXP
- U2 pad J2: unconnected-(U2G-USB30_RXP-PadJ2) -> /USB/USB3_RXP
- U2 pad J3: unconnected-(U2G-USB30_RXN-PadJ3) -> /USB/USB3_RXN
- U2 pad K1: unconnected-(U2G-USB30_DP-PadK1) -> /USB/USB3_DP
- U2 pad K2: unconnected-(U2G-USB30_DM-PadK2) -> /USB/USB3_DM
- U2 pad K7: unconnected-(U2G-USB30_VBUS-PadK7) -> VSYS
- U2 pad N1: unconnected-(U2H-CODEC_AOR-PadN1) -> /Audio/AUDIO_R
- U2 pad P2: unconnected-(U2H-CODEC_AOL-PadP2) -> /Audio/AUDIO_L
- U2 pad T4: unconnected-(U2H-CODEC_VCM-PadT4) -> Net-(U2H-CODEC_VCM)
- U2 pad T6: unconnected-(U2G-USB20_VBUS-PadT6) -> VSYS
- U2 pad U3: unconnected-(U2D-GPIO0_A4/HDMI_HPD-PadU3) -> /HDMI/HDMI_HPD
- U2 pad V1: unconnected-(U2D-I2C3_SCL/HDMI_SCL-PadV1) -> /HDMI/HDMI_SCL
- U2 pad V10: /main/SD_DETN -> unconnected-(U2F-GPIO1_A5/SDMMC0_DETN-PadV10)
- U2 pad V2: unconnected-(U2D-HDMI_CEC-PadV2) -> /HDMI/HDMI_CEC
- U2 pad V3: unconnected-(U2D-I2C3_SDA/HDMI_SDA-PadV3) -> /HDMI/HDMI_SDA
- U2 pad W2: unconnected-(U2D-HDMI_TXCLKN-PadW2) -> /HDMI/HDMI_CLKN
- U2 pad W6: unconnected-(U2G-USB20_EXTR-PadW6) -> Net-(U2G-USB20_EXTR)
- U2 pad Y1: unconnected-(U2D-HDMI_TXCLKP-PadY1) -> /HDMI/HDMI_CLKP
- U2 pad Y2: unconnected-(U2D-HDMI_TX0N-PadY2) -> /HDMI/HDMI_TX0N
- U2 pad Y3: unconnected-(U2D-HDMI_TX1N-PadY3) -> /HDMI/HDMI_TX1N
- U2 pad Y4: unconnected-(U2D-HDMI_TX1P-PadY4) -> /HDMI/HDMI_TX1P
- U2 pad Y5: unconnected-(U2D-HDMI_TX2P-PadY5) -> /HDMI/HDMI_TX2P
- U2 pad Y6: unconnected-(U2G-USB0_DM-PadY6) -> /USB/USB2_0_DM
- U2 pad Y7: unconnected-(U2G-USB1_DM-PadY7) -> /USB/USB2_1_DM
Routing:
- net /HDMI/HDMI_TX2P: track 0.00 -> 40.0 mm
- net /HDMI/HDMI_TX1P: track 0.00 -> 39.9 mm
- net /HDMI/HDMI_TX0N: track 0.00 -> 39.5 mm, vias 0 -> 2
- net /HDMI/HDMI_CLKN: track 0.00 -> 39.5 mm, vias 0 -> 2
- net /HDMI/HDMI_TX0P: track 0.00 -> 39.4 mm, vias 0 -> 2
- net /HDMI/HDMI_TX1N: track 0.00 -> 39.2 mm
- net /HDMI/HDMI_CLKP: track 0.00 -> 39.0 mm, vias 0 -> 2
- net /HDMI/HDMI_TX2N: track 0.00 -> 38.7 mm
- net Net-(J2-CEC): track 0.00 -> 19.0 mm, vias 0 -> 2
- net (no net): track 18.4 -> 0.00 mm, vias 3 -> 0
- net Net-(U1-VREFCA): track 0.00 -> 18.2 mm, vias 0 -> 2
- net /HDMI/HDMI_SDA: track 0.00 -> 17.8 mm
- net /HDMI/HDMI_HPD: track 0.00 -> 17.8 mm
- net Net-(J2-SCL): track 0.00 -> 16.8 mm
- net /HDMI/HDMI_CEC: track 0.00 -> 16.6 mm, vias 0 -> 2
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Other:
- board text added: "ADDRESS and CONTROL: 26.5 mm Both Data Lanes: 21 mm HDMI Diffrential pairs: 40 mm"
- board text removed: "ADDRESS and CONTROL: 26.5 mm Both Data Lanes: 21 mm"
