File: hardware/mini-server.kicad_pcb (KiCad board)
At the start: 6 copper layers, 85 x 55 mm, 111 parts, among them J1 RJ45_Hanrun_HR911105A_Horizon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, J2 HDMI_A, J3 Micro_SD_Card, J4 Conn_01x04_Pin, J5 AudioJack4, J6 USB_C_Receptacle, J7 USB_C_Receptacle, J8 USB_C_Receptacle, J9 USB_C_Receptacle, Q1 2N7002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

Commit message: routing
Parts:
- added C69: 22u, Capacitor_SMD:C_0603_1608Metric, F.Cu at (83.9, 106.3)
- added C70: 100n, Capacitor_SMD:C_0201_0603Metric, F.Cu at (108.9, 112.6)
- added C71: 100n, Capacitor_SMD:C_0201_0603Metric, F.Cu at (72.5, 113.9)
- added C72: C, Capacitor_SMD:C_0201_0603Metric, F.Cu at (107.1, 109.5)
- added C73: C, Capacitor_SMD:C_0201_0603Metric, F.Cu at (103.5, 109.5)
- added L6: 2.2u, Inductor_SMD:L_1008_2520Metric, F.Cu at (53.3, 93.8)
- added R16: R, Resistor_SMD:R_0201_0603Metric, F.Cu at (54.6, 106.7)
- added R17: R, Resistor_SMD:R_0201_0603Metric, F.Cu at (53.9, 107.8)
- added R18: R, Resistor_SMD:R_0201_0603Metric, F.Cu at (101.7, 116.2)
- added R19: R, Resistor_SMD:R_0201_0603Metric, F.Cu at (109.9, 114.6)
- added R20: R, Resistor_SMD:R_0201_0603Metric, F.Cu at (108.8, 116.1)
- added R21: 10m, Resistor_SMD:R_0402_1005Metric, F.Cu at (109.7, 112.6)
- added R22: 100, Resistor_SMD:R_0201_0603Metric, F.Cu at (69.9, 111.5)
- added R23: 100, Resistor_SMD:R_0201_0603Metric, F.Cu at (69.9, 110.8)
- added R24: 100, Resistor_SMD:R_0201_0603Metric, F.Cu at (69.9, 112.2)
- added R25: 100, Resistor_SMD:R_0201_0603Metric, B.Cu at (73.2, 110.1)
- added R26: 10k, Resistor_SMD:R_0201_0603Metric, F.Cu at (109.9, 113.9)
- added R27: 5.1k, Resistor_SMD:R_0201_0603Metric, F.Cu at (104.4, 116.5)
- added R28: R, Resistor_SMD:R_0201_0603Metric, F.Cu at (106.0, 109.1)
- added R29: R, Resistor_SMD:R_0201_0603Metric, F.Cu at (104.6, 109.1)
- added U10: BQ29209DRBR, Package_SON:VSON-8-1EP_3x3mm_P0.65mm_EP1.6x2.4mm, F.Cu at (73.2, 111.8)
- C62: moved to B.Cu
- U5: value BQ25690RBAR_C53283868 -> BQ25690RBAR
- moved L3 37.6 mm to (140.6, 85.1)
- moved R8 37.6 mm to (140.6, 82.6)
- moved R9 37.6 mm to (139.7, 81.1)
- moved C43 37.6 mm to (137.7, 84.8)
- moved C45 37.6 mm to (137.7, 83.3)
- moved C47 37.6 mm to (138.5, 82.2)
- moved C51 37.6 mm to (142.6, 86.7)
- moved U8 37.6 mm to (140.6, 81.7)
- moved C49 37.6 mm to (143.4, 85.6)
- moved L5 32.0 mm to (47.9, 105.6), turned to 180 degrees
- moved U5 30.9 mm to (105.3, 112.9)
- moved C66 30.8 mm to (48.8, 108.4), turned to -90 degrees
- moved C65 23.6 mm to (48.0, 101.7)
- moved U4 23.2 mm to (52.2, 105.9)
- moved C63 23.2 mm to (58.1, 98.8)
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Connections:
- C66 pad 1: Net-(U4-EN) -> /Power/BUCK_VIN
- C67 pad 1: Net-(U4-EN) -> /Power/BUCK_VIN
- C68 pad 1: Net-(U4-EN) -> /Power/BUCK_VIN
- U4 pad 3: Net-(U4-EN) -> /Power/BUCK_VIN
- U4 pad 5: Net-(U4-EN) -> /Power/BUCK_VIN
- U5 pad 1: unconnected-(U5-BTST1-Pad1) -> Net-(U5-BTST1)
- U5 pad 10: unconnected-(U5-GND-Pad10) -> GND
- U5 pad 11: unconnected-(U5-SCL-Pad11) -> PWR_SCL
- U5 pad 12: unconnected-(U5-SDA-Pad12) -> PWR_SDA
- U5 pad 13: unconnected-(U5-CELL-Pad13) -> Net-(BT1-+)
- U5 pad 14: unconnected-(U5-VCHG-Pad14) -> Net-(U5-VCHG)
- U5 pad 15: unconnected-(U5-ICHG-Pad15) -> Net-(U5-ICHG)
- U5 pad 16: unconnected-(U5-TS-Pad16) -> Net-(U5-TS)
- U5 pad 17: unconnected-(U5-SRN-Pad17) -> Net-(U5-SRN)
- U5 pad 18: unconnected-(U5-SRP-Pad18) -> Net-(Q2-S)
- U5 pad 19: unconnected-(U5-BATDRV-Pad19) -> Net-(Q2-G)
- U5 pad 20: unconnected-(U5-BTST2-Pad20) -> Net-(U5-BTST2)
- U5 pad 21: unconnected-(U5-SYS-Pad21) -> /Power/BUCK_VIN
- U5 pad 22: unconnected-(U5-SW2-Pad22) -> Net-(U5-SW2)
- U5 pad 23: unconnected-(U5-GND-Pad23) -> GND
- U5 pad 24: unconnected-(U5-SW1-Pad24) -> Net-(U5-SW1)
- U5 pad 25: unconnected-(U5-VIN-Pad25) -> VBUS
- U5 pad 26: unconnected-(U5-GND-Pad26) -> GND
- U5 pad 4: unconnected-(U5-ACN-Pad4) -> VBUS
- U5 pad 5: unconnected-(U5-ACP-Pad5) -> VBUS
- U5 pad 7: unconnected-(U5-ILIM_HIZ-Pad7) -> Net-(U5-ILIM_HIZ)
- U5 pad 8: unconnected-(U5-INT-Pad8) -> PWR_INT
- U5 pad 9: unconnected-(U5-~{CE}-Pad9) -> ~{PWR_CE}
Routing:
- net +1V8: track 3.67 -> 19.5 mm, vias 10 -> 13
- net +3V3: track 11.5 -> 22.9 mm
- net GND: track 169.1 -> 177.7 mm, vias 53 -> 66
- net Net-(U2E-GPIO1_B3/UART0_CTSN/GMAC_RXD0_M1): track 8.78 -> 17.0 mm
- net /Power/BUCK_VIN: track 0.00 -> 6.04 mm, vias 0 -> 3
- net VBUS: track 6.53 -> 11.9 mm, vias 0 -> 4
- net Net-(U2E-GPIO1_B2/UART0_RTSN/GMAC_RXD1_M1): track 10.9 -> 15.6 mm
- net Net-(U2H-CODEC_VCM): track 0.06 -> 4.67 mm, vias 1 -> 2
- net /USB/USB2_0_D+: track 47.8 -> 52.2 mm, vias 2 -> 3
- net Net-(U10-VDD): track 0.00 -> 3.27 mm, vias 0 -> 1
- net Net-(U5-ICHG): track 0.00 -> 2.81 mm
- net Net-(U5-TS): track 0.00 -> 2.70 mm
- net Net-(Q2-S): track 0.00 -> 2.67 mm
- net Net-(U5-SRN): track 0.00 -> 2.67 mm
- net VSYS: track 13.4 -> 16.0 mm, vias 2 -> 1
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- added copper zone on In3.Cu, net +1V0
- added copper zone on In3.Cu, net +1V8
- added copper zone on In3.Cu, net +3V3
- added copper zone on F.Cu, net VBUS
- removed copper zone on In3.Cu, net GND

Commit message: routing and power pours
Parts:
- moved C66 57.8 mm to (106.6, 109.3), turned to 0 degrees
- moved L5 55.3 mm to (103.2, 106.8)
- moved R16 55.0 mm to (109.6, 108.1)
- moved C62 55.0 mm to (106.9, 106.8)
- moved U4 55.0 mm to (107.2, 106.9)
- moved R17 54.9 mm to (108.8, 109.2)
- moved C68 54.5 mm to (104.4, 108.5), turned to 180 degrees
- moved C64 54.2 mm to (101.9, 108.5)
- moved C67 53.8 mm to (104.4, 109.2), turned to 180 degrees
- moved C65 53.6 mm to (101.6, 104.7), turned to 90 degrees
- moved L6 53.2 mm to (101.9, 115.4), turned to -90 degrees
- moved C63 45.7 mm to (103.4, 104.7)
- moved R24 42.6 mm to (112.2, 117.3), turned to -90 degrees
- moved R22 42.0 mm to (111.5, 117.3), turned to -90 degrees
- moved R23 41.4 mm to (110.8, 117.3), turned to -90 degrees
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Routing:
- net unconnected-(J3-SHIELD-PadSH): track 0.00 -> 30.2 mm, vias 0 -> 2
- net VSYS: track 16.0 -> 39.3 mm, vias 1 -> 42
- net +3V3: track 22.9 -> 31.2 mm, vias 16 -> 17
- net VBUS: track 11.9 -> 6.60 mm, vias 4 -> 0
- net Net-(U5-SW1): track 2.46 -> 0.00 mm
- net Net-(U4-FB): track 0.00 -> 2.42 mm
- net Net-(U5-SW2): track 2.41 -> 0.01 mm
- net Net-(BT1-+): track 1.86 -> 3.68 mm
- net /Power/BUCK_VIN: track 6.04 -> 4.46 mm, vias 3 -> 6
- net Net-(U10-CD): track 0.00 -> 1.52 mm
- net Net-(U5-VCHG): track 2.03 -> 2.85 mm
- net GND: track 177.7 -> 178.3 mm
- net Net-(U5-ILIM_HIZ): track 2.16 -> 1.60 mm
- added copper zone on F.Cu, net /Power/BUCK_VIN
- added copper zone on In3.Cu, net /Power/BUCK_VIN
- added copper zone on F.Cu, net Net-(U5-SW1)
- added copper zone on F.Cu, net Net-(U5-SW2)
- added copper zone on F.Cu, net VSYS
- added copper zone on In3.Cu, net VSYS

Commit message: touch up on lots of small things
Parts:
- added BT1: Battery_Cell, Connector_JST:JST_XH_B2B-XH-AM_1x02_P2.50mm_Vertical, F.Cu at (100.4, 100.2)
- added BT2: Battery_Cell, Connector_JST:JST_XH_B2B-XH-AM_1x02_P2.50mm_Vertical, F.Cu at (100.4, 91.8)
- added C74: 100n, Capacitor_SMD:C_0201_0603Metric, F.Cu at (116.4, 119.6)
- added C75: 100n, Capacitor_SMD:C_0201_0603Metric, F.Cu at (115.7, 119.6)
- added D1: LED, LED_SMD:LED_0402_1005Metric, F.Cu at (99.1, 113.2)
- added R30: 10k, Resistor_SMD:R_0201_0603Metric, F.Cu at (142.0, 87.9)
- added R31: 10k, Resistor_SMD:R_0201_0603Metric, F.Cu at (142.3, 81.6)
- added R32: 10k, Resistor_SMD:R_0201_0603Metric, F.Cu at (112.2, 78.4)
- added R33: 10k, Resistor_SMD:R_0201_0603Metric, F.Cu at (116.3, 102.2)
- added R34: 100, Resistor_SMD:R_0201_0603Metric, F.Cu at (99.1, 111.1)
- C62, R25, R6, R7: moved to F.Cu
- R27: value 5.1k -> 10k
- moved R27 16.9 mm to (122.4, 106.5), turned to 135 degrees
- moved C54 3.49 mm to (159.2, 94.9)
- moved J1 3.49 mm to (164.5, 101.9)
- moved C53 3.49 mm to (159.2, 98.8)
- moved J5 2.46 mm to (131.8, 120.5)
- moved C62 2.14 mm to (106.0, 104.9)
- moved R6 2.07 mm to (108.9, 78.3)
- moved C57 1.91 mm to (132.8, 113.5), turned to 0 degrees
- moved C56 1.68 mm to (129.6, 113.5), turned to 0 degrees
- moved R23 1.68 mm to (109.7, 116.0), turned to 90 degrees
- moved R7 1.64 mm to (108.2, 78.3), turned to -90 degrees
- moved R25 0.53 mm to (109.7, 114.2)
- moved J6 0.25 mm to (118.5, 124.9)
- moved J9 0.25 mm to (107.8, 124.9)
- moved C28 0.22 mm to (136.2, 99.4), turned to 180 degrees
Connections:
- J6 pad A2: /USB/USB3_TXP -> Net-(J6-TX1+)
- J6 pad A3: /USB/USB3_TXN -> Net-(J6-TX1-)
- U1 pad J1: unconnected-(U1-NC-PadJ1) -> GND
- U2 pad D1: unconnected-(U2H-GPIO3_A5/TSP_D1/CIF_D1/SDMMC0EXT_D1/UART1_RTSN/USB3PHY_DEBUG5-PadD1) -> ~{PWR_CE}
- U2 pad D2: unconnected-(U2H-GPIO3_A1/TSP_FAIL/CIF_HREF/SDMMC0EXT_DET/SPI_TXD_M2/USB3PHY_DEBUG2/I2S2_SDO_M1-PadD2) -> PWR_INT
- U2 pad N19: unconnected-(U2H-GPIO2_A4/PWM0/I2C1_SDA-PadN19) -> PWR_SDA
- U2 pad N20: unconnected-(U2H-GPIO2_A5/PWM1/I2C1_SCL-PadN20) -> PWR_SCL
- U2 pad P21: unconnected-(U2H-NPOR-PadP21) -> NPOR
- U6 pad 4: unconnected-(U6-PG-Pad4) -> Net-(U6-PG)
- U7 pad 4: unconnected-(U7-PG-Pad4) -> Net-(U7-PG)
- U7 pad 5: unconnected-(U7-EN-Pad5) -> Net-(U6-PG)
- U8 pad 4: unconnected-(U8-PG-Pad4) -> Net-(U8-PG)
- U8 pad 5: unconnected-(U8-EN-Pad5) -> Net-(U7-PG)
- U9 pad 4: unconnected-(U9-PG-Pad4) -> NPOR
- U9 pad 5: unconnected-(U9-EN-Pad5) -> Net-(U8-PG)
Routing:
- net PWR_SDA: track 1.34 -> 46.1 mm, vias 1 -> 2
- net PWR_SCL: track 1.10 -> 44.1 mm, vias 1 -> 2
- net Net-(U8-PG): track 0.00 -> 41.7 mm, vias 0 -> 2
- net NPOR: track 0.00 -> 40.2 mm, vias 0 -> 2
- net Net-(U6-PG): track 0.00 -> 37.0 mm
- net PWR_INT: track 1.14 -> 35.2 mm, vias 1 -> 0
- net ~{PWR_CE}: track 1.68 -> 33.8 mm, vias 1 -> 0
- net Net-(U7-PG): track 0.00 -> 31.1 mm
- net VSYS: track 39.3 -> 56.8 mm, vias 42 -> 48
- net GND: track 178.3 -> 188.6 mm, vias 66 -> 112
- net +3V3: track 31.2 -> 39.8 mm, vias 17 -> 19
- net Net-(BT1--): track 0.70 -> 8.70 mm, vias 0 -> 2
- net VBUS: track 6.60 -> 0.06 mm
- net /USB/USB3_D+: track 28.0 -> 31.9 mm
- net /Ethernet/PHY_DATA_LED: track 43.0 -> 39.0 mm
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- added copper zone on B.Cu, net Net-(BT1-+)
- added copper zone on F.Cu, net Net-(BT1-+)
- added copper zone on B.Cu, net Net-(BT1--)
- added copper zone on F.Cu, net Net-(U4-SW)
Other:
- board text added: "ADDRESS and CONTROL: 26.5 mm Both Data Lanes: 21 mm HDMI Diffrential pairs: 27.7381 mm"
- board text removed: "ADDRESS and CONTROL: 26.5 mm Both Data Lanes: 21 mm HDMI Diffrential pairs: 27.8 mm"
