File: hardware/Power.kicad_sch (KiCad schematic)
At the start: 1 part, among them U2 RK3328

Commit message: stuff
Parts:
- removed U2: RK3328, easyeda2kicad:TFBGA395_L14.0-W14.0_RK3328, symbol easyeda2kicad:RK3328
- added C20, C34, C36, C38, C39, C41, C43, C44, C45, C46, C49, C50: 10u, Capacitor_SMD:C_0603_1608Metric, symbol Device:C
- added C35, C37, C40, C42, C47, C48, C51, C52: 100n, Capacitor_SMD:C_0201_0603Metric, symbol Device:C_Small
- added L1, L2, L3, L4: 2.2u, Inductor_SMD:L_1008_2520Metric, symbol Device:L
- added Q1: 2N7002, Package_TO_SOT_SMD:SOT-23, symbol Transistor_FET:2N7002
- added R10, R11, R12, R4, R5, R6, R7, R8, R9: R, Resistor_SMD:R_0201_0603Metric, symbol Device:R_Small
- added U6, U7, U8, U9: TPS563252DRLR, easyeda2kicad:SOT-563-6_L1.6-W1.2-P0.50-LS1.6-BL, symbol easyeda2kicad:TPS563252DRLR
Connections:
- net +1V5: now also C41.1, C42.1, L2.2
- net GND: now also C20.2, C34.2, C35.2, C36.2, C37.2, C38.2, C39.2, C40.2, C41.2, C42.2, C43.2, C44.2, C45.2, C46.2, C47.2, C48.2, C49.2, C50.2, C51.2, C52.2, Q1.2 (S), R11.2, R5.2, R7.2, R9.2, U6.3 (GND), U7.3 (GND), U8.3 (GND), U9.3 (GND)
- new net: L3.1, R8.1, U8.2 (SW)
- new net: R8.2, R9.1, U8.6 (FB)
- new net: R12.1, R4.2, R5.1, U6.6 (FB)
- new net: Q1.3 (D), R12.2
- new net: L2.1, R6.1, U7.2 (SW)
- new net: R6.2, R7.1, U7.6 (FB)
- new net: L4.1, R10.1, U9.2 (SW)
- new net: L1.1, R4.1, U6.2 (SW)
- new net: R10.2, R11.1, U9.6 (FB)
- new net +1V0: C36.1, C37.1, L1.2
- new net +1V8: C49.1, C51.1, L3.2
- new net +3V3: C50.1, C52.1, L4.2
- new net VSYS: C20.1, C34.1, C35.1, C38.1, C39.1, C40.1, C43.1, C44.1, C45.1, C46.1, C47.1, C48.1, U6.1 (VIN), U6.5 (EN), U7.1 (VIN), U8.1 (VIN), U9.1 (VIN)
Other:
- added sheet RK3328 Symbols (Power_rk3328.kicad_sch)
- note added: "Power On Sequence: +1v0 -> +1v5 -> +1v8 -> +3v3"

Commit message: Routing and PCB
Other:
- note added: "VSYS is the internal 5v"
Changed lines of the file:
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@@
+		)
+	)
+	(text "VSYS is the internal 5v"
+		(exclude_from_sim no)
+		(at 99.822 52.07 0)
+		(effects
+			(font
+				(size 1.27 1.27)
+			)
 		)
 	)

Commit message: component Placement
Parts:
- added U4: BQ25887RGE, Package_DFN_QFN:Texas_RGE0024H_VQFN-24-1EP_4x4mm_P0.5mm_EP2.7x2.7mm, symbol Battery_Management:BQ25887RGE
Connections:
- net GND: now also U4.19 (GND), U4.20 (GND), U4.25 (GND)
- new net: U4.13 (BAT), U4.14 (BAT)
- new net: U4.15 (SNS), U4.16 (SNS)
- new net: U4.17 (SW), U4.18 (SW)
- new net: U4.21 (PMID), U4.22 (PMID)
Changed lines of the file:
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@@
 	(wire
 		(pts
+			(xy 256.54 166.37) (xy 256.54 167.64)
+		)
+		(stroke
+			(width 0)
+			(type default)
+		)
+	)
+	(wire
+		(pts
 			(xy 109.22 121.92) (xy 119.38 121.92)
 		)
@@
 	)
 	(symbol
+		(lib_id "power:GND")
+		(at 256.54 167.64 0)
+		(unit 1)
+		(body_style 1)
+		(exclude_from_sim no)
+		(in_bom yes)
+		(on_board yes)
+		(in_pos_files yes)
+		(dnp no)
+		(fields_autoplaced yes)
+		(property "Reference" "#PWR077"
+			(at 256.54 173.99 0)
+			(hide yes)
+			(show_name no)
+			(do_not_autoplace no)
+			(effects
+				(font
+					(size 1.27 1.27)
+				)
+			)
+		)
+		(property "Value" "GND"
+			(at 256.54 172.72 0)
+			(show_name no)
+			(do_not_autoplace no)
+			(effects
+				(font
+					(size 1.27 1.27)
+				)
+			)
+		)
+		(property "Footprint" ""
+			(at 256.54 167.64 0)
+			(hide yes)
+			(show_name no)
+			(do_not_autoplace no)
+			(effects
+				(font
+					(size 1.27 1.27)
+				)
+			)
+		)
+		(property "Datasheet" ""
+			(at 256.54 167.64 0)
+			(hide yes)
+			(show_name no)
+			(do_not_autoplace no)
+			(effects
+				(font
+					(size 1.27 1.27)
+				)
+			)
+		)
+		(property "Description" "Power symbol creates a global label with name \"GND\" , ground"
+			(at 256.54 167.64 0)
+			(hide yes)
+			(show_name no)
+			(do_not_autoplace no)
+			(effects
+				(font
+					(size 1.27 1.27)
+				)
+			)
+		)
+		(pin "1"
+		)
+		(instances
+			(project "mini-server"
+				(path "/17ecef2a-4000-49de-93ef-dcbfcfdaa69f/3600fbf6-de14-44f9-b86f-9b010ddcaaed"
+					(reference "#PWR077")
+					(unit 1)
+				)
+			)
+		)
+	)
+	(symbol
 		(lib_id "Device:C")
 		(at 64.77 160.02 0)
@@
 					(unit 1)
 				)
+			)
+		)
+	)
+	(symbol
+		(lib_id "Battery_Management:BQ25887RGE")
+		(at 256.54 143.51 0)
+		(unit 1)
+		(body_style 1)
+		(exclude_from_sim no)
+		(in_bom yes)
+		(on_board yes)
+		(in_pos_files yes)
+		(dnp no)
+		(fields_autoplaced yes)
+		(property "Reference" "U4"
+			(at 256.54 118.11 0)
+			(show_name no)
+			(do_not_autoplace no)
+			(effects
+				(font
+					(size 1.27 1.27)
+				)
+			)
+		)
+		(property "Value" "BQ25887RGE"
+			(at 256.54 120.65 0)
+			(show_name no)
+			(do_not_autoplace no)
+			(effects
+				(font
+					(size 1.27 1.27)
+				)
+			)
+		)
+		(property "Footprint" "Package_DFN_QFN:Texas_RGE0024H_VQFN-24-1EP_4x4mm_P0.5mm_EP2.7x2.7mm"
+			(at 256.54 172.974 0)
+			(hide yes)
+			(show_name no)
+			(do_not_autoplace no)
+			(effects
+				(font
+					(size 1.27 1.27)
+				)
+			)
+		)
+		(property "Datasheet" "https://www.ti.com/lit/ds/symlink/bq25887.pdf"
+			(at 256.54 170.942 0)
+			(hide yes)
+			(show_name no)
+			(do_not_autoplace no)
+			(effects
+				(font
+					(size 1.27 1.27)
+				)
+			)
+		)
+		(property "Description" "I2C Controlled 2-Cell (Li-Ion / Li-Polymer), 2A boost-mode battery charger with cell balancing for USB input, 3.9..6.2V VBUS, 3.4..4.6V charge voltage regulation range (per cell), 1.5 MHz, VQFN-24"
+			(at 256.54 168.91 0)
+			(hide yes)
+			(show_name no)
+			(do_not_autoplace no)
+			(effects
+				(font
+					(size 1.27 1.27)
+				)
+			)
+		)
+		(pin "3"
+		)
+		(pin "23"
+		)
+		(pin "10"
+		)
+		(pin "6"
+		)
+		(pin "4"
+		)
+		(pin "12"
+		)
+		(pin "20"
+		)
+		(pin "13"
+		)
+		(pin "8"
+		)
+		(pin "9"
+		)
+		(pin "2"
+		)
+		(pin "15"
+		)
+		(pin "17"
+		)
+		(pin "19"
+		)
+		(pin "21"
+		)
+		(pin "18"
+		)
+		(pin "24"
+		)
+		(pin "22"
+		)
+		(pin "25"
+		)
+		(pin "7"
+		)
+		(pin "5"
+		)
+		(pin "1"
+		)
+		(pin "16"
+		)
+		(pin "11"
+		)
+		(pin "14"
+		)
+		(instances
+			(project "mini-server"
+				(path "/17ecef2a-4000-49de-93ef-dcbfcfdaa69f/3600fbf6-de14-44f9-b86f-9b010ddcaaed"
+					(reference "U4")
+					(unit 1)
+				)

Commit message: routing
Parts:
- added BT1, BT2: Battery_Cell, symbol Device:Battery_Cell
- added C62: C_Small, symbol Device:C_Small
- added J9: USB_C_Receptacle, Connector_USB:USB_C_Receptacle_Molex_105450-0101, symbol Connector:USB_C_Receptacle
Connections:
- net GND: now also J9.A1 (GND), J9.A12 (GND), J9.B1 (GND), J9.B12 (GND), J9.SH (SHIELD); no longer C49.2, C51.2
- net at U4.11 (REGN): now also C62.1
- net at U4.13 (BAT), U4.14 (BAT): now also BT1.1 (+)
- net at U4.23 (VBUS): now also J9.A4 (VBUS), J9.A9 (VBUS), J9.B4 (VBUS), J9.B9 (VBUS)
- net at U4.9 (MID): now also BT1.2 (-), BT2.1 (+)
- new net: C49.2, C51.2
- no-connect marks 0 -> 14
Other:
- moved on the sheet: U4

Commit message: New battery charger IC
Parts:
- removed U4: BQ25887RGE, Package_DFN_QFN:Texas_RGE0024H_VQFN-24-1EP_4x4mm_P0.5mm_EP2.7x2.7mm, symbol Battery_Management:BQ25887RGE
- added C63, C66: 10u, Capacitor_SMD:C_0603_1608Metric, symbol Device:C
- added C64, C67: 100n, Capacitor_SMD:C_0201_0603Metric, symbol Device:C_Small
- added C65, C68: 1u, Capacitor_SMD:C_0201_0603Metric, symbol Device:C_Small
- added C69: 22u, symbol Device:C
- added L5: 2.2u, Inductor_SMD:L_1008_2520Metric, symbol Device:L
- added R16, R17: R, symbol Device:R_Small
- added U4: TPS565201, Package_TO_SOT_SMD:SOT-23-6, symbol Regulator_Switching:TPS565201
- added U5: BQ25690RBAR_C53283868, easyeda2kicad:WQFN-26_L4.0-W3.5_BQ25690RBAR, symbol easyeda2kicad:BQ25690RBAR_C53283868
- C62: value C_Small -> 100n; footprint (none) -> Capacitor_SMD:C_0201_0603Metric
Connections:
- net GND: now also BT2.2 (-), C49.2, C51.2, C63.2, C64.2, C65.2, C66.2, C67.2, C68.2, C69.2, R17.2, U4.1 (GND), U5.10 (GND), U5.23 (GND), U5.26 (GND)
- net VSYS: now also C63.1, C64.1, C65.1, C69.1, L5.2, R16.1
- net at BT1.1 (+): now also U5.13 (CELL)
- net at C62.1: now also U4.6 (VBST)
- net at C62.2: now also L5.1, U4.2 (SW)
- net VBUS: now reaches J9.A4 (VBUS), J9.A9 (VBUS), J9.B4 (VBUS), J9.B9 (VBUS)
- net VBUS: now also U5.25 (VIN)
- new net: C66.1, C67.1, C68.1, U4.3 (VIN), U4.5 (EN)
- new net: R16.2, R17.1, U4.4 (FB)
- new net PWR_SCL: U5.11 (SCL)
- new net PWR_SDA: U5.12 (SDA)
Other:
- moved on the sheet: BT1, BT2, C20, C34, C35, C36, C37, C38, C39, C40, C41, C42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

Commit message: routing
Parts:
- added C70, C71: 100n, Capacitor_SMD:C_0201_0603Metric, symbol Device:C_Small
- added C72, C73: C, Capacitor_SMD:C_0201_0603Metric, symbol Device:C_Small
- added L6: 2.2u, Inductor_SMD:L_1008_2520Metric, symbol Device:L
- added Q2: NMOS, symbol Simulation_SPICE:NMOS
- added R18, R19, R20, R28, R29: R, Resistor_SMD:R_0201_0603Metric, symbol Device:R_Small
- added R21: 10m, Resistor_SMD:R_0402_1005Metric, symbol Device:R_Small
- added R22, R23, R24, R25: 100, Resistor_SMD:R_0201_0603Metric, symbol Device:R_Small
- added R26: 10k, Resistor_SMD:R_0201_0603Metric, symbol Device:R_Small
- added R27: 5.1k, Resistor_SMD:R_0201_0603Metric, symbol Device:R_Small
- added U10: BQ29209DRBR, Package_SON:VSON-8-1EP_3x3mm_P0.65mm_EP1.6x2.4mm, symbol easyeda2kicad:BQ29209DRBR
- C69: footprint (none) -> Capacitor_SMD:C_0603_1608Metric
- R16, R17: footprint (none) -> Resistor_SMD:R_0201_0603Metric
- U5: value BQ25690RBAR_C53283868 -> BQ25690RBAR
Connections:
- net GND: now also C71.2, R18.2, R19.2, R20.2, R26.1, R27.2, U10.5 (GND), U10.6 (~{CB_EN}), U10.9 (EP)
- net VBUS: now also U5.4 (ACN), U5.5 (ACP)
- net BUCK_VIN: now reaches C66.1, C67.1, C68.1, U4.3 (VIN), U4.5 (EN)
- net BUCK_VIN: now also U5.21 (SYS), Q2.1 (D)
- net at BT1.1 (+), U5.13 (CELL): now also R23.2, R25.2
- net at BT1.2 (-), BT2.1 (+): now also R22.2, R24.2
- net at U5.1 (BTST1): now also C73.1
- net at U5.14 (VCHG): now also R20.1
- net at U5.15 (ICHG): now also R19.1
- net at U5.16 (TS): now also R26.2
- net at U5.17 (SRN): now also C70.2, R21.2
- net at U5.18 (SRP): now also C70.1, Q2.3 (S), R21.1
- net at U5.19 (BATDRV): now also Q2.2 (G)
- net at U5.20 (BTST2): now also C72.1
- net at U5.22 (SW2): now also L6.1, R28.2
- net at U5.24 (SW1): now also L6.2, R29.2
- net at U5.7 (ILIM_HIZ): now also R18.1
- net PWR_INT: now reaches U5.8 (INT)
- net ~{PWR_CE}: now reaches U5.9 (~{CE})
- net ~{PWR_CE}: now also R27.1
- new net: R24.1, U10.3 (VC1_CB)
- new net: C72.2, R28.1
- new net: C73.2, R29.1
- new net: R25.1, U10.7 (VDD)
- new net: R23.1, U10.1 (VC2)
- new net: R22.1, U10.2 (VC1)
- new net: C71.1, U10.4 (CD)
- no-connect marks 14 -> 15
Other:
- moved on the sheet: BT1, BT2, U5

Commit message: touch up on lots of small things
Parts:
- added D1: LED, LED_SMD:LED_0402_1005Metric, symbol Device:LED
- added R30, R31, R32, R33: 10k, Resistor_SMD:R_0201_0603Metric, symbol Device:R_Small
- added R34: 100, Resistor_SMD:R_0201_0603Metric, symbol Device:R_Small
- BT1, BT2: footprint (none) -> Connector_JST:JST_XH_B2B-XH-AM_1x02_P2.50mm_Vertical
- R27: value 5.1k -> 10k
Connections:
- net +3V3: now also R30.2
- net GND: now also R34.2
- net VSYS: now also D1.2 (A), R31.2, R32.2, R33.2
- net at U6.4 (PG): now also U7.5 (EN), R33.1
- net at U7.4 (PG): now also U8.5 (EN), R32.1
- net NPOR: now reaches U9.4 (PG)
- net NPOR: now also R30.1
- net at U9.5 (EN): now also U8.4 (PG), R31.1
- new net: D1.1 (K), R34.1

Commit message: final touches
Parts:
- removed R10, R7: R, Resistor_SMD:R_0201_0603Metric, symbol Device:R_Small
- added R35, R38, R40: 10k, Resistor_SMD:R_0201_0603Metric, symbol Device:R_Small
- added R36, R37: 5.1k, Resistor_SMD:R_0201_0603Metric, symbol Device:R
- added R39: 5.1k, Resistor_SMD:R_0201_0603Metric, symbol Device:R_Small
- added R41: 35k, Resistor_SMD:R_0201_0603Metric, symbol Device:R_Small
- added TP3, TP4, TP5, TP6, TP7, TP8, TP9: TestPoint, TestPoint:TestPoint_Pad_D1.0mm, symbol Connector:TestPoint
- C72, C73: value C -> 47n
- Q2: value NMOS -> AON7262e; footprint (none) -> easyeda2kicad:DFN-8_L3.3-W3.3-P0.65-BL
- R11, R17, R5, R6, R8, R9: value R -> 10k
- R12: value R -> 35k
- R16: value R -> 56k
- R28, R29: value R -> 0R
- R4: value R -> 6.6k
Connections:
- net +1V0: now also R4.1, TP3.1
- net +1V5: now also R38.1, TP4.1
- net +1V8: now also R8.1, TP5.1
- net +3V3: now also R41.1, TP6.1
- net BUCK_VIN: now also Q2.5 (D), TP8.1; no longer Q2.1 (D)
- net GND: now also R36.2, R37.2, R40.2
- net VBUS: now also TP9.1
- net VSYS: now also TP7.1
- net at L3.1, U8.2 (SW): no longer R8.1
- net at R9.1, U8.6 (FB): now also R35.2; no longer R8.2
- net at C70.1, Q2.3 (S), R21.1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: now also Q2.1 (S), Q2.2 (S)
- net at L2.1, U7.2 (SW): no longer R6.1
- net at U7.6 (FB): now also R39.2, R40.1; no longer R6.2
- net at L1.1, U6.2 (SW): no longer R4.1
- net at U5.19 (BATDRV): now also Q2.4 (G); no longer Q2.2 (G)
- net PWR_CTRL: now reaches Q1.1 (G)
- net at R11.1, U9.6 (FB): now also R6.2
- net CC1: now reaches J9.A5 (CC1)
- net CC1: now also R37.1
- net CC2: now reaches J9.B5 (CC2)
- net CC2: now also R36.1
- new net: R38.2, R39.1
- new net: R35.1, R8.2
- new net: R41.2, R6.1
Other:
- moved on the sheet: C36, C37, Q1, R11, R12, R16, R17, R30, R4, R5
