File: hardware/Power.kicad_sch (KiCad schematic)
At the start: 91 parts, among them J9 USB_C_Receptacle, Q1 2N7002, Q2 AON7262e, U10 BQ29209DRBR, U4 TPS565201, U5 BQ25690RBAR, U6 TPS563252DRLR, U7 TPS563252DRLR, U8 TPS563252DRLR, U9 TPS563252DRLR

Commit message: resistor values fixed
Parts:
- removed C69: 22u, Capacitor_SMD:C_0603_1608Metric, symbol Device:C
Changed lines of the file:
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@@
 	)
 	(junction
-		(at 248.92 259.08)
-		(diameter 0)
-		(color 0 0 0 0)
-	)
-	(junction
 		(at 241.3 254)
 		(diameter 0)
@@
 	)
 	(junction
-		(at 256.54 254)
-		(diameter 0)
-		(color 0 0 0 0)
-	)
-	(junction
 		(at 356.87 154.94)
 		(diameter 0)
@@
 	(wire
 		(pts
-			(xy 256.54 254) (xy 270.51 254)
-		)
-		(stroke
-			(width 0)
-			(type default)
-		)
-	)
-	(wire
-		(pts
 			(xy 189.23 191.77) (xy 177.8 191.77)
 		)
@@
 	(wire
 		(pts
-			(xy 256.54 261.62) (xy 248.92 261.62)
-		)
-		(stroke
-			(width 0)
-			(type default)
-		)
-	)
-	(wire
-		(pts
 			(xy 356.87 115.57) (xy 361.95 115.57)
 		)
@@
 	(wire
 		(pts
-			(xy 248.92 261.62) (xy 248.92 259.08)
-		)
-		(stroke
-			(width 0)
-			(type default)
-		)
-	)
-	(wire
-		(pts
 			(xy 344.17 195.58) (xy 347.98 195.58)
 		)
@@
 	(wire
 		(pts
-			(xy 248.92 254) (xy 256.54 254)
+			(xy 248.92 254) (xy 270.51 254)
 		)
 		(stroke
@@
 					(unit 1)
 				)
-			)
-		)
-	)
-	(symbol
-		(lib_id "Device:C")
-		(at 256.54 257.81 0)
-		(unit 1)
-		(body_style 1)
-		(exclude_from_sim no)
-		(in_bom yes)
-		(on_board yes)
-		(in_pos_files yes)
-		(dnp no)
-		(fields_autoplaced yes)
-		(property "Reference" "C69"
-			(at 260.35 256.5399 0)
-			(show_name no)
-			(do_not_autoplace no)
-			(effects
-				(font
-					(size 1.27 1.27)
-				)
-				(justify left)
-			)
-		)
-		(property "Value" "22u"
-			(at 260.35 259.0799 0)
-			(show_name no)
-			(do_not_autoplace no)
-			(effects
-				(font
-					(size 1.27 1.27)
-				)
-				(justify left)
-			)
-		)
-		(property "Footprint" "Capacitor_SMD:C_0603_1608Metric"
-			(at 257.5052 261.62 0)
-			(hide yes)
-			(show_name no)
-			(do_not_autoplace no)
-			(effects
-				(font
-					(size 1.27 1.27)
-				)
-			)
-		)
-		(property "Datasheet" ""
-			(at 256.54 257.81 0)
-			(hide yes)
-			(show_name no)
-			(do_not_autoplace no)
-			(effects
-				(font
-					(size 1.27 1.27)
-				)
-			)
-		)
-		(property "Description" "Unpolarized capacitor"
-			(at 256.54 257.81 0)
-			(hide yes)
-			(show_name no)
-			(do_not_autoplace no)
-			(effects
-				(font
-					(size 1.27 1.27)
-				)
-			)
-		)
-		(pin "2"
-		)
-		(pin "1"
-		)
-		(instances
-			(project "mini-server"
-				(path "/17ecef2a-4000-49de-93ef-dcbfcfdaa69f/3600fbf6-de14-44f9-b86f-9b010ddcaaed"
-					(reference "C69")
-					(unit 1)
-				)
