File: hardware/Power_rk3328.kicad_sch (KiCad schematic)
At the start: 14 parts, among them U2 RK3328

Commit message: routing
Connections:
- net +3V3: now also U2.H6 (VCCIO6), U2.R16 (VCCIO5), U2.T17 (VCCIO2), U2.U12 (VCCIO4), U2.U7 (VCCIO3)
Changed lines of the file:
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@@
+	)
+	(junction
+		(at 176.53 101.6)
+		(diameter 0)
+		(color 0 0 0 0)
 	)
 	(junction
@@
 	)
 	(junction
+		(at 176.53 106.68)
+		(diameter 0)
+		(color 0 0 0 0)
+	)
+	(junction
 		(at 374.65 147.32)
 		(diameter 0)
@@
 	)
 	(junction
+		(at 176.53 109.22)
+		(diameter 0)
+		(color 0 0 0 0)
+	)
+	(junction
 		(at 306.07 104.14)
 		(diameter 0)
@@
 	)
 	(junction
+		(at 176.53 99.06)
+		(diameter 0)
+		(color 0 0 0 0)
+	)
+	(junction
 		(at 306.07 38.1)
 		(diameter 0)
@@
 	)
 	(junction
+		(at 176.53 104.14)
+		(diameter 0)
+		(color 0 0 0 0)
+	)
+	(junction
 		(at 50.8 198.12)
 		(diameter 0)
@@
 	(wire
 		(pts
+			(xy 176.53 99.06) (xy 176.53 101.6)
+		)
+		(stroke
+			(width 0)
+			(type default)
+		)
+	)
+	(wire
+		(pts
 			(xy 306.07 96.52) (xy 306.07 99.06)
 		)
@@
 	(wire
 		(pts
+			(xy 176.53 101.6) (xy 176.53 104.14)
+		)
+		(stroke
+			(width 0)
+			(type default)
+		)
+	)
+	(wire
+		(pts
 			(xy 76.2 113.03) (xy 76.2 116.84)
 		)
@@
 	(wire
 		(pts
+			(xy 176.53 106.68) (xy 176.53 109.22)
+		)
+		(stroke
+			(width 0)
+			(type default)
+		)
+	)
+	(wire
+		(pts
 			(xy 77.47 68.58) (xy 90.17 68.58)
 		)
@@
 	(wire
 		(pts
+			(xy 176.53 104.14) (xy 176.53 106.68)
+		)
+		(stroke
+			(width 0)
+			(type default)
+		)
+	)
+	(wire
+		(pts
 			(xy 374.65 220.98) (xy 374.65 223.52)
 		)
@@
 	(wire
 		(pts
+			(xy 90.17 129.54) (xy 69.85 129.54)
+		)
+		(stroke
+			(width 0)
+			(type default)
+		)
+	)
+	(wire
+		(pts
 			(xy 90.17 105.41) (xy 90.17 107.95)
 		)
@@
 	(wire
 		(pts
+			(xy 69.85 125.73) (xy 69.85 129.54)
+		)
+		(stroke
+			(width 0)
+			(type default)
+		)
+	)
+	(wire
+		(pts
 			(xy 306.07 134.62) (xy 306.07 137.16)
 		)
@@
 		)
 		(stroke
+			(width 0)
+			(type default)
+		)
+	)
+	(wire
+		(pts
+			(xy 176.53 109.22) (xy 176.53 111.76)
+		)
+		(stroke

Commit message: final touches
Parts:
- added TP10: TestPoint, TestPoint:TestPoint_Pad_D1.0mm, symbol Connector:TestPoint
Connections:
- net +1V0: now also U2.M5 (VDD_PMU)
- net +1V8: now also U2.N16 (OTP_VCC18)
- net GND: now also TP10.1
Changed lines of the file:
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@@
 	)
 	(junction
+		(at 87.63 124.46)
+		(diameter 0)
+		(color 0 0 0 0)
+	)
+	(junction
 		(at 306.07 48.26)
 		(diameter 0)
@@
 	)
 	(junction
+		(at 374.65 231.14)
+		(diameter 0)
+		(color 0 0 0 0)
+	)
+	(junction
 		(at 306.07 45.72)
 		(diameter 0)
@@
 	)
 	(junction
+		(at 76.2 134.62)
+		(diameter 0)
+		(color 0 0 0 0)
+	)
+	(junction
 		(at 374.65 93.98)
 		(diameter 0)
@@
 	(wire
 		(pts
-			(xy 76.2 121.92) (xy 76.2 139.7)
+			(xy 76.2 121.92) (xy 76.2 134.62)
 		)
 		(stroke
@@
 	(wire
 		(pts
+			(xy 90.17 134.62) (xy 76.2 134.62)
+		)
+		(stroke
+			(width 0)
+			(type default)
+		)
+	)
+	(wire
+		(pts
 			(xy 90.17 110.49) (xy 87.63 110.49)
 		)
@@
 	(wire
 		(pts
+			(xy 87.63 129.54) (xy 90.17 129.54)
+		)
+		(stroke
+			(width 0)
+			(type default)
+		)
+	)
+	(wire
+		(pts
 			(xy 374.65 190.5) (xy 374.65 193.04)
 		)
@@
 	(wire
 		(pts
+			(xy 374.65 231.14) (xy 377.19 231.14)
+		)
+		(stroke
+			(width 0)
+			(type default)
+		)
+	)
+	(wire
+		(pts
 			(xy 306.07 38.1) (xy 306.07 40.64)
 		)
@@
 	(wire
 		(pts
+			(xy 87.63 124.46) (xy 87.63 129.54)
+		)
+		(stroke
+			(width 0)
+			(type default)
+		)
+	)
+	(wire
+		(pts
 			(xy 374.65 220.98) (xy 374.65 223.52)
 		)
@@
 	(wire
 		(pts
-			(xy 90.17 129.54) (xy 69.85 129.54)
-		)
-		(stroke
-			(width 0)
-			(type default)
-		)
-	)
-	(wire
-		(pts
 			(xy 90.17 105.41) (xy 90.17 107.95)
 		)
@@
 	(wire
 		(pts
-			(xy 69.85 125.73) (xy 69.85 129.54)
-		)
-		(stroke
-			(width 0)
-			(type default)
-		)
-	)
-	(wire
-		(pts
 			(xy 306.07 134.62) (xy 306.07 137.16)
 		)
@@
 	(wire
 		(pts
+			(xy 76.2 134.62) (xy 76.2 139.7)
+		)
+		(stroke
+			(width 0)
+			(type default)
+		)
+	)
+	(wire
+		(pts
 			(xy 306.07 121.92) (xy 306.07 124.46)
 		)
@@
 				)
 			)
+		)
+	)
+	(symbol
+		(lib_id "Connector:TestPoint")
+		(at 377.19 231.14 0)
+		(unit 1)
+		(body_style 1)
+		(exclude_from_sim no)
+		(in_bom yes)
+		(on_board yes)
+		(in_pos_files yes)
+		(dnp no)
+		(fields_autoplaced yes)
+		(property "Reference" "TP10"
+			(at 379.73 226.5679 0)
+			(show_name no)
+			(do_not_autoplace no)
+			(effects
+				(font
+					(size 1.27 1.27)
+				)
+				(justify left)
+			)
+		)
+		(property "Value" "TestPoint"
+			(at 379.73 229.1079 0)
+			(hide yes)
+			(show_name no)
+			(do_not_autoplace no)
+			(effects
+				(font
+					(size 1.27 1.27)
+				)
+				(justify left)
+			)
+		)
+		(property "Footprint" "TestPoint:TestPoint_Pad_D1.0mm"
+			(at 382.27 231.14 0)
+			(hide yes)
+			(show_name no)
+			(do_not_autoplace no)
+			(effects
+				(font
+					(size 1.27 1.27)
+				)
+			)
+		)
+		(property "Datasheet" ""
+			(at 382.27 231.14 0)
+			(hide yes)
+			(show_name no)
+			(do_not_autoplace no)
+			(effects
+				(font
+					(size 1.27 1.27)
+				)
+			)
+		)
+		(property "Description" "test point"
+			(at 377.19 231.14 0)
+			(hide yes)
+			(show_name no)
+			(do_not_autoplace no)
+			(effects
+				(font
+					(size 1.27 1.27)
+				)
+			)
+		)
+		(pin "1"
+		)
+		(instances
+			(project "mini-server"
+				(path "/17ecef2a-4000-49de-93ef-dcbfcfdaa69f/3600fbf6-de14-44f9-b86f-9b010ddcaaed/66b52930-0c85-4676-845f-af1d7e666d61"
+					(reference "TP10")
+					(unit 1)
+				)
+			)
