File: hardware/main.kicad_sch (KiCad schematic)
At the start: 1 part, among them U2 RK3328

Commit message: stuff
Parts:
- added R13: R, symbol Device:R
Connections:
- net PHY_RXN: now reaches U2.AA8 (FEPHY_RXN)
- net PHY_TXN: now reaches U2.AA9 (FEPHY_TXN)
- net at U2.V7 (FEPHY_EXTRES): now also R13.1
- net PHY_RXP: now reaches U2.Y8 (FEPHY_RXP)
- net PHY_TXP: now reaches U2.Y9 (FEPHY_TXP)
- net SD_DAT3: now reaches U2.AA13 (GPIO1_A3/SDMMC0_D3/JTAG_TMS)
- net SD_DAT0: now reaches U2.U10 (GPIO1_A0/SDMMC0_D0/UART2_TX_M0)
- net SD_DETN: now reaches U2.V10 (GPIO1_A5/SDMMC0_DETN)
- net SD_DAT1: now reaches U2.W11 (GPIO1_A1/SDMMC0_D1/UART2_RX_M0)
- net SD_CLK: now reaches U2.W12 (GPIO1_A6/SDMMC0_CLK/TEST_CLK0)
- net SD_DAT2: now reaches U2.W13 (GPIO1_A2/SDMMC0_D2/JTAG_TCK)
- net SD_CMD: now reaches U2.Y13 (GPIO1_A4/SDMMC0_CMD)
- new net GND: R13.2
- new net PHY_DATA_LED: U2.R17 (GPIO2_D1/I2C0_SDA/FEPHY_LED_DATA_M1)
- new net PHY_LINK_LED: U2.P17 (GPIO2_D0/I2C0_SCL/FEPHY_LED_LINK_M1)

Commit message: Routing and PCB
Parts:
- added C59: 10u, Capacitor_SMD:C_0603_1608Metric, symbol Device:C_Small
- added R14, R15: R, symbol Device:R
Connections:
- net GND: now also C59.1, R14.2, R15.2
- net AUDIO_R: now reaches U2.N1 (CODEC_AOR)
- net AUDIO_L: now reaches U2.P2 (CODEC_AOL)
- net at U2.T4 (CODEC_VCM): now also C59.2
- net USB2_0_DP: now reaches U2.AA6 (USB0_DP)
- net USB2_1_DP: now reaches U2.AA7 (USB1_DP)
- net at U2.G5 (USB30_EXTR): now also R14.1
- net USB3_TXN: now reaches U2.H2 (USB30_TXN)
- net USB3_TXP: now reaches U2.H3 (USB30_TXP)
- net USB3_RXP: now reaches U2.J2 (USB30_RXP)
- net USB3_RXN: now reaches U2.J3 (USB30_RXN)
- net USB3_DP: now reaches U2.K1 (USB30_DP)
- net USB3_DM: now reaches U2.K2 (USB30_DM)
- net VSYS: now reaches U2.K7 (USB30_VBUS)
- net VSYS: now also U2.T6 (USB20_VBUS)
- net at U2.W6 (USB20_EXTR): now also R15.1
- net USB2_0_DM: now reaches U2.Y6 (USB0_DM)
- net USB2_1_DM: now reaches U2.Y7 (USB1_DM)
- net HDMI_TX0P: now reaches U2.AA2 (HDMI_TX0P)
- net HDMI_TX2N: now reaches U2.AA4 (HDMI_TX2N)
- net HDMI_HPD: now reaches U2.U3 (GPIO0_A4/HDMI_HPD)
- net HDMI_SCL: now reaches U2.V1 (I2C3_SCL/HDMI_SCL)
- net HDMI_CEC: now reaches U2.V2 (HDMI_CEC)
- net HDMI_SDA: now reaches U2.V3 (I2C3_SDA/HDMI_SDA)
- net HDMI_CLKN: now reaches U2.W2 (HDMI_TXCLKN)
- net HDMI_CLKP: now reaches U2.Y1 (HDMI_TXCLKP)
- net HDMI_TX0N: now reaches U2.Y2 (HDMI_TX0N)
- net HDMI_TX1N: now reaches U2.Y3 (HDMI_TX1N)
- net HDMI_TX1P: now reaches U2.Y4 (HDMI_TX1P)
- net HDMI_TX2P: now reaches U2.Y5 (HDMI_TX2P)
- net SD_DAT0 renamed SD_D0
- net SD_DAT1 renamed SD_D1
- net SD_DAT2 renamed SD_D2
- net SD_DAT3 renamed SD_D3
- net SD_DETN: no longer names the net of U2.V10 (GPIO1_A5/SDMMC0_DETN)
- no-connect marks 24 -> 25

Commit message: component Placement
Parts:
- added C60, C61: C_Small, symbol Device:C_Small
- added J4: Conn_01x04_Pin, symbol Connector:Conn_01x04_Pin
- added TP1: ~{UART0_CTS}, symbol Connector:TestPoint
- added TP2: ~{UART0_RST}, symbol Connector:TestPoint
- added Y1: Crystal_GND24, symbol Device:Crystal_GND24
Connections:
- net GND: now also C60.2, C61.2, J4.4 (Pin_4)
- net at U2.R1 (XIN24M): now also C60.1, Y1.3
- net at U2.T1 (XOUT24M): now also C61.1, Y1.1
- net at U2.AA15 (GPIO1_B1/UART0_TX/GMAC_TXD0_M1): now also J4.2 (Pin_2)
- net at U2.V13 (GPIO1_B3/UART0_CTSN/GMAC_RXD0_M1): now also TP1.1
- net at U2.W14 (GPIO1_B2/UART0_RTSN/GMAC_RXD1_M1): now also TP2.1
- net at U2.Y15 (GPIO1_B0/UART0_RX/GMAC_TXD1_M1): now also J4.3 (Pin_3)
- net USB2_0_DM renamed USB2_0_D-
- net USB2_0_DP renamed USB2_0_D+
- net USB2_1_DM renamed USB2_1_D-
- net USB2_1_DP renamed USB2_1_D+
- new net: Y1.2 (G), Y1.4 (G)
- no-connect marks 25 -> 54
Other:
- note added: "Connect PWR here"

Commit message: routing
Parts:
- C60, C61: footprint (none) -> Capacitor_SMD:C_0201_0603Metric
- J4: footprint (none) -> Connector_PinHeader_2.54mm:PinHeader_1x04_P2.54mm_Vertical
- R13, R14, R15: footprint (none) -> Resistor_SMD:R_0201_0603Metric
- TP1, TP2: footprint (none) -> TestPoint:TestPoint_Pad_D1.0mm
- Y1: footprint (none) -> Crystal:Crystal_SMD_3225-4Pin_3.2x2.5mm
Connections:
- net GND: now also Y1.2 (G), Y1.4 (G)
- net at C60.1, U2.R1 (XIN24M): now also Y1.1; no longer Y1.3
- net at C61.1, U2.T1 (XOUT24M): now also Y1.3; no longer Y1.1
- net USB3_DM renamed USB3_D-
- net USB3_DP renamed USB3_D+
- no-connect marks 54 -> 66
Other:
- moved on the sheet: Y1
Changed lines of the file:
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@@
 	)
 	(junction
-		(at 394.97 259.08)
+		(at 394.97 276.86)
 		(diameter 0)
 		(color 0 0 0 0)
 	)
 	(junction
-		(at 394.97 276.86)
+		(at 394.97 259.08)
 		(diameter 0)
 		(color 0 0 0 0)
@@
 	)
 	(no_connect
+		(at 92.71 326.39)
+	)
+	(no_connect
 		(at 191.77 121.92)
 	)
@@
 	)
 	(no_connect
+		(at 92.71 316.23)
+	)
+	(no_connect
 		(at 191.77 124.46)
 	)
@@
 	)
 	(no_connect
+		(at 92.71 318.77)
+	)
+	(no_connect
 		(at 417.83 330.2)
 	)
@@
 	)
 	(no_connect
+		(at 92.71 311.15)
+	)
+	(no_connect
 		(at 105.41 104.14)
 	)
 	(no_connect
+		(at 275.59 336.55)
+	)
+	(no_connect
 		(at 417.83 335.28)
 	)
@@
 	)
 	(no_connect
+		(at 92.71 308.61)
+	)
+	(no_connect
 		(at 191.77 104.14)
 	)
@@
 	)
 	(no_connect
+		(at 92.71 323.85)
+	)
+	(no_connect
 		(at 140.97 241.3)
 	)
 	(no_connect
+		(at 92.71 321.31)
+	)
+	(no_connect
 		(at 105.41 133.35)
 	)
@@
 	)
 	(no_connect
+		(at 92.71 300.99)
+	)
+	(no_connect
 		(at 191.77 116.84)
 	)
@@
 	)
 	(no_connect
+		(at 92.71 306.07)
+	)
+	(no_connect
 		(at 351.79 311.15)
 	)
@@
 	)
 	(no_connect
+		(at 92.71 303.53)
+	)
+	(no_connect
 		(at 537.21 334.01)
 	)
@@
 	)
 	(no_connect
+		(at 92.71 313.69)
+	)
+	(no_connect
 		(at 105.41 127)
 	)
@@
 		)
 	)
+	(wire
+		(pts
+			(xy 400.05 262.89) (xy 401.32 262.89)
+		)
+		(stroke
+			(width 0)
+			(type default)
+		)
+	)
 	(bus
 		(pts
@@
 	(wire
 		(pts
-			(xy 394.97 276.86) (xy 394.97 266.7)
-		)
-		(stroke
-			(width 0)
-			(type default)
-		)
-	)
-	(wire
-		(pts
 			(xy 248.92 341.63) (xy 248.92 340.36)
 		)
@@
 		)
 	)
+	(wire
+		(pts
+			(xy 401.32 262.89) (xy 401.32 264.16)
+		)
+		(stroke
+			(width 0)
+			(type default)
+		)
+	)
 	(bus
 		(pts
@@
 		)
 	)
+	(wire
+		(pts
+			(xy 394.97 266.7) (xy 394.97 276.86)
+		)
+		(stroke
+			(width 0)
+			(type default)
+		)
+	)
 	(bus
 		(pts
@@
 		)
 	)
-	(label "USB3_DM"
-		(at 200.66 259.08 0)
-		(effects
-			(font
-				(size 1.27 1.27)
-			)
-			(justify left bottom)
-		)
-	)
 	(label "{FEPHY}"
 		(at 259.08 325.12 270)
@@
 		)
 	)
-	(label "USB3_DP"
-		(at 200.66 256.54 0)
-		(effects
-			(font
-				(size 1.27 1.27)
-			)
-			(justify left bottom)
-		)
-	)
 	(label "HDMI_TX2N"
 		(at 77.47 237.49 0)
@@
 		)
 	)
+	(label "USB3_D+"
+		(at 209.55 256.54 180)
+		(effects
+			(font
+				(size 1.27 1.27)
+			)
+			(justify right bottom)
+		)
+	)
 	(label "DQL1"
 		(at 198.12 53.34 0)
@@
 		)
 	)
+	(label "USB3_D-"
+		(at 209.55 259.08 180)
+		(effects
+			(font
+				(size 1.27 1.27)
+			)
+			(justify right bottom)
+		)
+	)
 	(label "USB2_1_D-"
 		(at 262.89 259.08 0)
@@
 			)
 		)
-		(property "Footprint" ""
+		(property "Footprint" "TestPoint:TestPoint_Pad_D1.0mm"
 			(at 372.11 300.99 0)
 			(hide yes)
@@
 			)
 		)
-		(property "Footprint" ""
+		(property "Footprint" "TestPoint:TestPoint_Pad_D1.0mm"
 			(at 365.76 295.91 0)
 			(hide yes)
@@
 			)
 		)
-		(property "Footprint" ""
+		(property "Footprint" "Resistor_SMD:R_0201_0603Metric"
 			(at 201.422 267.97 90)
 			(hide yes)
@@
 			)
 		)
-		(property "Footprint" ""
+		(property "Footprint" "Resistor_SMD:R_0201_0603Metric"
 			(at 247.142 336.55 90)
 			(hide yes)
@@
 			)
 		)
-		(property "Footprint" ""
+		(property "Footprint" "Capacitor_SMD:C_0201_0603Metric"
 			(at 394.97 279.4 0)
 			(hide yes)
@@
 	(symbol
 		(lib_id "Device:Crystal_GND24")
-		(at 394.97 262.89 270)
+		(at 394.97 262.89 90)
 		(unit 1)
 		(body_style 1)
@@
 		(fields_autoplaced yes)
 		(property "Reference" "Y1"
-			(at 400.05 261.6199 90)
+			(at 389.89 261.6199 90)
 			(show_name no)
 			(do_not_autoplace no)
@@
 		)
 		(property "Value" "Crystal_GND24"
-			(at 400.05 264.1599 90)
+			(at 389.89 264.1599 90)
 			(show_name no)
 			(do_not_autoplace no)
@@
 			)
 		)
-		(property "Footprint" ""
+		(property "Footprint" "Crystal:Crystal_SMD_3225-4Pin_3.2x2.5mm"
 			(at 394.97 262.89 0)
 			(hide yes)
@@
 		)
 		(property private "KLC_S3.3" "The rectangle is not a symbol body but a graphical element"
-			(at 382.27 262.89 0)
+			(at 407.67 262.89 0)
 			(hide yes)
 			(show_name yes)
@@
 		)
 		(property private "KLC_S4.1" "Some pins are on 50mil grid to make the symbol small"
-			(at 379.73 262.89 0)
+			(at 410.21 262.89 0)
 			(hide yes)
 			(show_name yes)
@@
 			)
 		)
-		(property "Footprint" ""
+		(property "Footprint" "Resistor_SMD:R_0201_0603Metric"
 			(at 262.382 267.97 90)
 			(hide yes)
@@
 	)
 	(symbol
+		(lib_id "power:GND")
+		(at 401.32 264.16 0)
+		(unit 1)
+		(body_style 1)
+		(exclude_from_sim no)
+		(in_bom yes)
+		(on_board yes)
+		(in_pos_files yes)
+		(dnp no)
+		(fields_autoplaced yes)
+		(property "Reference" "#PWR078"
+			(at 401.32 270.51 0)
+			(hide yes)
+			(show_name no)
+			(do_not_autoplace no)
+			(effects
+				(font
+					(size 1.27 1.27)
+				)
+			)
+		)
+		(property "Value" "GND"
+			(at 401.32 269.24 0)
+			(show_name no)
+			(do_not_autoplace no)
+			(effects
+				(font
+					(size 1.27 1.27)
+				)
+			)
+		)
+		(property "Footprint" ""
+			(at 401.32 264.16 0)
+			(hide yes)
+			(show_name no)
+			(do_not_autoplace no)
+			(effects
+				(font
+					(size 1.27 1.27)
+				)
+			)
+		)
+		(property "Datasheet" ""
+			(at 401.32 264.16 0)
+			(hide yes)
+			(show_name no)
+			(do_not_autoplace no)
+			(effects
+				(font
+					(size 1.27 1.27)
+				)
+			)
+		)
+		(property "Description" "Power symbol creates a global label with name \"GND\" , ground"
+			(at 401.32 264.16 0)
+			(hide yes)
+			(show_name no)
+			(do_not_autoplace no)
+			(effects
+				(font
+					(size 1.27 1.27)
+				)
+			)
+		)
+		(pin "1"
+		)
+		(instances
+			(project "mini-server"
+				(path "/17ecef2a-4000-49de-93ef-dcbfcfdaa69f/385b9ec2-ad34-4f97-be56-79080b11a749"
+					(reference "#PWR078")
+					(unit 1)
+				)
+			)
+		)
+	)
+	(symbol
 		(lib_id "Connector:Conn_01x04_Pin")
 		(at 378.46 316.23 0)
@@
 			)
 		)
-		(property "Footprint" ""
+		(property "Footprint" "Connector_PinHeader_2.54mm:PinHeader_1x04_P2.54mm_Vertical"
 			(at 378.46 316.23 0)
 			(hide yes)
@@
 			)
 		)
-		(property "Footprint" ""
+		(property "Footprint" "Capacitor_SMD:C_0201_0603Metric"
 			(at 381 257.81 0)
 			(hide yes)

Commit message: touch up on lots of small things
Connections:
- net ~{PWR_CE}: now reaches U2.D1 (GPIO3_A5/TSP_D1/CIF_D1/SDMMC0EXT_D1/UART1_RTSN/USB3PHY_DEBUG5)
- net PWR_INT: now reaches U2.D2 (GPIO3_A1/TSP_FAIL/CIF_HREF/SDMMC0EXT_DET/SPI_TXD_M2/USB3PHY_DEBUG2/I2S2_SDO_M1)
- net PWR_SDA: now reaches U2.N19 (GPIO2_A4/PWM0/I2C1_SDA)
- net PWR_SCL: now reaches U2.N20 (GPIO2_A5/PWM1/I2C1_SCL)
- net NPOR: now reaches U2.P21 (NPOR)
Changed lines of the file:
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@@
+	(wire
+		(pts
+			(xy 537.21 311.15) (xy 541.02 311.15)
+		)
+		(stroke
+			(width 0)
+			(type default)
+		)
+	)
 	(wire
 		(pts
@@
 		)
 	)
+	(wire
+		(pts
+			(xy 537.21 308.61) (xy 541.02 308.61)
+		)
+		(stroke
+			(width 0)
+			(type default)
+		)
+	)
 	(bus
 		(pts
@@
 	(wire
 		(pts
+			(xy 537.21 306.07) (xy 541.02 306.07)
+		)
+		(stroke
+			(width 0)
+			(type default)
+		)
+	)
+	(wire
+		(pts
 			(xy 77.47 242.57) (xy 92.71 242.57)
 		)
@@
 	(wire
 		(pts
+			(xy 537.21 321.31) (xy 541.02 321.31)
+		)
+		(stroke
+			(width 0)
+			(type default)
+		)
+	)
+	(wire
+		(pts
 			(xy 97.79 147.32) (xy 105.41 147.32)
 		)
@@
 		(pts
 			(xy 191.77 73.66) (xy 205.74 73.66)
+		)
+		(stroke
+			(width 0)
+			(type default)
+		)
+	)
+	(wire
+		(pts
+			(xy 415.29 279.4) (xy 417.83 279.4)
 		)
 		(stroke
@@
 		)
 	)
+	(global_label "PWR_SCL"
+		(shape input)
+		(at 541.02 308.61 0)
+		(fields_autoplaced yes)
+		(effects
+			(font
+				(size 1.27 1.27)
+			)
+			(justify left)
+		)
+		(property "Intersheetrefs" "${INTERSHEET_REFS}"
+			(at 552.4718 308.61 0)
+			(hide yes)
+			(show_name no)
+			(do_not_autoplace no)
+			(effects
+				(font
+					(size 1.27 1.27)
+				)
+				(justify left)
+			)
+		)
+	)
+	(global_label "~{PWR_CE}"
+		(shape input)
+		(at 537.21 290.83 0)
+		(fields_autoplaced yes)
+		(effects
+			(font
+				(size 1.27 1.27)
+			)
+			(justify left)
+		)
+		(property "Intersheetrefs" "${INTERSHEET_REFS}"
+			(at 547.5732 290.83 0)
+			(hide yes)
+			(show_name no)
+			(do_not_autoplace no)
+			(effects
+				(font
+					(size 1.27 1.27)
+				)
+				(justify left)
+			)
+		)
+	)
+	(global_label "PWR_SDA"
+		(shape input)
+		(at 541.02 306.07 0)
+		(fields_autoplaced yes)
+		(effects
+			(font
+				(size 1.27 1.27)
+			)
+			(justify left)
+		)
+		(property "Intersheetrefs" "${INTERSHEET_REFS}"
+			(at 552.5323 306.07 0)
+			(hide yes)
+			(show_name no)
+			(do_not_autoplace no)
+			(effects
+				(font
+					(size 1.27 1.27)
+				)
+				(justify left)
+			)
+		)
+	)
+	(global_label "PWR_INT"
+		(shape input)
+		(at 537.21 288.29 0)
+		(fields_autoplaced yes)
+		(effects
+			(font
+				(size 1.27 1.27)
+			)
+			(justify left)
+		)
+		(property "Intersheetrefs" "${INTERSHEET_REFS}"
+			(at 548.0571 288.29 0)
+			(hide yes)
+			(show_name no)
+			(do_not_autoplace no)
+			(effects
+				(font
+					(size 1.27 1.27)
+				)
+				(justify left)
+			)
+		)
+	)
+	(global_label "NPOR"
+		(shape input)
+		(at 415.29 279.4 180)
+		(fields_autoplaced yes)
+		(effects
+			(font
+				(size 1.27 1.27)
+			)
+			(justify right)
+		)
+		(property "Intersheetrefs" "${INTERSHEET_REFS}"
+			(at 407.1038 279.4 0)
+			(hide yes)
+			(show_name no)
+			(do_not_autoplace no)
+			(effects
+				(font
+					(size 1.27 1.27)
+				)
+				(justify right)
+			)
+		)
+	)

Commit message: final touches
Parts:
- added TP11: TestPoint, TestPoint:TestPoint_Pad_D1.0mm, symbol Connector:TestPoint
Connections:
- net PWR_CTRL: now reaches U2.E1 (GPIO3_A2/TSP_CLK/CIF_CLKIN/SDMMC0EXT_CLK/SPI_RXD_M2/USB3PHY_DEBUG3/I2S2_SDI_M1)
- net at U2.N2 (GPIO_MUTE): now also TP11.1
- net +3V3: now reaches J4.1 (Pin_1)
Changed lines of the file:
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@@
 	(text "Connect PWR here"
 		(exclude_from_sim no)
-		(at 368.554 306.07 0)
+		(at 365.252 315.468 0)
 		(effects
 			(font
@@
 		)
 	)
+	(wire
+		(pts
+			(xy 417.83 297.18) (xy 408.94 297.18)
+		)
+		(stroke
+			(width 0)
+			(type default)
+		)
+	)
 	(bus
 		(pts
@@
 	(wire
 		(pts
-			(xy 537.21 311.15) (xy 541.02 311.15)
-		)
-		(stroke
-			(width 0)
-			(type default)
-		)
-	)
-	(wire
-		(pts
 			(xy 275.59 331.47) (xy 248.92 331.47)
 		)
@@
 	(wire
 		(pts
+			(xy 408.94 294.64) (xy 408.94 297.18)
+		)
+		(stroke
+			(width 0)
+			(type default)
+		)
+	)
+	(wire
+		(pts
 			(xy 101.6 73.66) (xy 105.41 73.66)
 		)
@@
 	(wire
 		(pts
-			(xy 537.21 321.31) (xy 541.02 321.31)
-		)
-		(stroke
-			(width 0)
-			(type default)
-		)
-	)
-	(wire
-		(pts
 			(xy 97.79 147.32) (xy 105.41 147.32)
 		)
@@
 		)
 	)
+	(global_label "PWR_CTRL"
+		(shape input)
+		(at 537.21 285.75 0)
+		(fields_autoplaced yes)
+		(effects
+			(font
+				(size 1.27 1.27)
+			)
+			(justify left)
+		)
+		(property "Intersheetrefs" "${INTERSHEET_REFS}"
+			(at 549.6899 285.75 0)
+			(hide yes)
+			(show_name no)
+			(do_not_autoplace no)
+			(effects
+				(font
+					(size 1.27 1.27)
+				)
+				(justify left)
+			)
+		)
+	)
 	(global_label "~{PWR_CE}"
 		(shape input)
@@
 	)
 	(symbol
+		(lib_id "power:+3V3")
+		(at 368.3 308.61 0)
+		(unit 1)
+		(body_style 1)
+		(exclude_from_sim no)
+		(in_bom yes)
+		(on_board yes)
+		(in_pos_files yes)
+		(dnp no)
+		(fields_autoplaced yes)
+		(property "Reference" "#PWR0101"
+			(at 368.3 312.42 0)
+			(hide yes)
+			(show_name no)
+			(do_not_autoplace no)
+			(effects
+				(font
+					(size 1.27 1.27)
+				)
+			)
+		)
+		(property "Value" "+3V3"
+			(at 368.3 303.53 0)
+			(show_name no)
+			(do_not_autoplace no)
+			(effects
+				(font
+					(size 1.27 1.27)
+				)
+			)
+		)
+		(property "Footprint" ""
+			(at 368.3 308.61 0)
+			(hide yes)
+			(show_name no)
+			(do_not_autoplace no)
+			(effects
+				(font
+					(size 1.27 1.27)
+				)
+			)
+		)
+		(property "Datasheet" ""
+			(at 368.3 308.61 0)
+			(hide yes)
+			(show_name no)
+			(do_not_autoplace no)
+			(effects
+				(font
+					(size 1.27 1.27)
+				)
+			)
+		)
+		(property "Description" "Power symbol creates a global label with name \"+3V3\""
+			(at 368.3 308.61 0)
+			(hide yes)
+			(show_name no)
+			(do_not_autoplace no)
+			(effects
+				(font
+					(size 1.27 1.27)
+				)
+			)
+		)
+		(pin "1"
+		)
+		(instances
+			(project "mini-server"
+				(path "/17ecef2a-4000-49de-93ef-dcbfcfdaa69f/385b9ec2-ad34-4f97-be56-79080b11a749"
+					(reference "#PWR0101")
+					(unit 1)
+				)
+			)
+		)
+	)
+	(symbol
 		(lib_id "Device:R")
 		(at 203.2 267.97 0)
@@
 				)
 			)
+		)
+	)
+	(symbol
+		(lib_id "Connector:TestPoint")
+		(at 408.94 294.64 0)
+		(unit 1)
+		(body_style 1)
+		(exclude_from_sim no)
+		(in_bom yes)
+		(on_board yes)
+		(in_pos_files yes)
+		(dnp no)
+		(fields_autoplaced yes)
+		(property "Reference" "TP11"
+			(at 411.48 290.0679 0)
+			(show_name no)
+			(do_not_autoplace no)
+			(effects
+				(font
+					(size 1.27 1.27)
+				)
+				(justify left)
+			)
+		)
+		(property "Value" "TestPoint"
+			(at 411.48 292.6079 0)
+			(hide yes)
+			(show_name no)
+			(do_not_autoplace no)
+			(effects
+				(font
+					(size 1.27 1.27)
+				)
+				(justify left)
+			)
+		)
+		(property "Footprint" "TestPoint:TestPoint_Pad_D1.0mm"
+			(at 414.02 294.64 0)
+			(hide yes)
+			(show_name no)
+			(do_not_autoplace no)
+			(effects
+				(font
+					(size 1.27 1.27)
+				)
+			)
+		)
+		(property "Datasheet" ""
+			(at 414.02 294.64 0)
+			(hide yes)
+			(show_name no)
+			(do_not_autoplace no)
+			(effects
+				(font
+					(size 1.27 1.27)
+				)
+			)
+		)
+		(property "Description" "test point"
+			(at 408.94 294.64 0)
+			(hide yes)
+			(show_name no)
+			(do_not_autoplace no)
+			(effects
+				(font
+					(size 1.27 1.27)
+				)
+			)
+		)
+		(pin "1"
+		)
+		(instances
+			(project "mini-server"
+				(path "/17ecef2a-4000-49de-93ef-dcbfcfdaa69f/385b9ec2-ad34-4f97-be56-79080b11a749"
+					(reference "TP11")
+					(unit 1)
+				)
+			)
