File: hardware/storage.kicad_sch (KiCad schematic)
At the start: 1 part, among them J3 Micro_SD_Card

Commit message: stuff
Parts:
- added C55: 100n, Capacitor_SMD:C_0201_0603Metric, symbol Device:C_Small
Connections:
- net SD_DAT2: now reaches J3.1 (DAT2)
- net SD_DAT3: now reaches J3.2 (DAT3/CD)
- net SD_CMD: now reaches J3.3 (CMD)
- net +3V3: now reaches J3.4 (VDD)
- net +3V3: now also C55.1
- net SD_CLK: now reaches J3.5 (CLK)
- net GND: now reaches J3.6 (VSS)
- net GND: now also C55.2
- net SD_DAT0: now reaches J3.7 (DAT0)
- net SD_DAT1: now reaches J3.8 (DAT1)

Commit message: Routing and PCB
Connections:
- net SD_DAT0 renamed SD_D0
- net SD_DAT1 renamed SD_D1
- net SD_DAT2 renamed SD_D2
- net SD_DAT3 renamed SD_D3
Changed lines of the file:
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@@
 	(paper "A4")
 	(bus_entry
-		(at 129.54 83.82)
-		(size 2.54 2.54)
-		(stroke
-			(width 0)
-			(type default)
-		)
-	)
-	(bus_entry
-		(at 129.54 91.44)
-		(size 2.54 2.54)
-		(stroke
-			(width 0)
-			(type default)
-		)
-	)
-	(bus_entry
-		(at 129.54 96.52)
-		(size 2.54 2.54)
-		(stroke
-			(width 0)
-			(type default)
-		)
-	)
-	(bus_entry
-		(at 129.54 86.36)
-		(size 2.54 2.54)
-		(stroke
-			(width 0)
-			(type default)
-		)
-	)
-	(bus_entry
-		(at 129.54 99.06)
-		(size 2.54 2.54)
-		(stroke
-			(width 0)
-			(type default)
-		)
-	)
-	(bus_entry
-		(at 129.54 81.28)
-		(size 2.54 2.54)
-		(stroke
-			(width 0)
-			(type default)
-		)
-	)
-	(wire
-		(pts
-			(xy 132.08 88.9) (xy 143.51 88.9)
+		(at 123.19 99.06)
+		(size 2.54 2.54)
+		(stroke
+			(width 0)
+			(type default)
+		)
+	)
+	(bus_entry
+		(at 123.19 86.36)
+		(size 2.54 2.54)
+		(stroke
+			(width 0)
+			(type default)
+		)
+	)
+	(bus_entry
+		(at 123.19 81.28)
+		(size 2.54 2.54)
+		(stroke
+			(width 0)
+			(type default)
+		)
+	)
+	(bus_entry
+		(at 123.19 91.44)
+		(size 2.54 2.54)
+		(stroke
+			(width 0)
+			(type default)
+		)
+	)
+	(bus_entry
+		(at 123.19 83.82)
+		(size 2.54 2.54)
+		(stroke
+			(width 0)
+			(type default)
+		)
+	)
+	(bus_entry
+		(at 123.19 96.52)
+		(size 2.54 2.54)
+		(stroke
+			(width 0)
+			(type default)
+		)
+	)
+	(wire
+		(pts
+			(xy 125.73 93.98) (xy 143.51 93.98)
+		)
+		(stroke
+			(width 0)
+			(type default)
+		)
+	)
+	(wire
+		(pts
+			(xy 125.73 86.36) (xy 143.51 86.36)
 		)
 		(stroke
@@
 	(bus
 		(pts
-			(xy 129.54 78.74) (xy 129.54 99.06)
-		)
-		(stroke
-			(width 0)
-			(type default)
-		)
-	)
-	(wire
-		(pts
-			(xy 132.08 99.06) (xy 143.51 99.06)
-		)
-		(stroke
-			(width 0)
-			(type default)
-		)
-	)
-	(wire
-		(pts
-			(xy 132.08 93.98) (xy 143.51 93.98)
+			(xy 123.19 78.74) (xy 123.19 101.6)
+		)
+		(stroke
+			(width 0)
+			(type default)
+		)
+	)
+	(wire
+		(pts
+			(xy 125.73 83.82) (xy 143.51 83.82)
+		)
+		(stroke
+			(width 0)
+			(type default)
+		)
+	)
+	(wire
+		(pts
+			(xy 125.73 99.06) (xy 143.51 99.06)
 		)
 		(stroke
@@
 	(wire
 		(pts
-			(xy 132.08 83.82) (xy 143.51 83.82)
+			(xy 125.73 101.6) (xy 143.51 101.6)
 		)
 		(stroke
@@
 	(wire
 		(pts
-			(xy 132.08 86.36) (xy 143.51 86.36)
-		)
-		(stroke
-			(width 0)
-			(type default)
-		)
-	)
-	(wire
-		(pts
 			(xy 140.97 91.44) (xy 143.51 91.44)
 		)
@@
 	(wire
 		(pts
-			(xy 132.08 101.6) (xy 143.51 101.6)
-		)
-		(stroke
-			(width 0)
-			(type default)
+			(xy 125.73 88.9) (xy 143.51 88.9)
+		)
+		(stroke
+			(width 0)
+			(type default)
+		)
+	)
+	(label "SD_D2"
+		(at 127 83.82 0)
+		(effects
+			(font
+				(size 1.27 1.27)
+			)
+			(justify left bottom)
+		)
+	)
+	(label "SD_CLK"
+		(at 127 93.98 0)
+		(effects
+			(font
+				(size 1.27 1.27)
+			)
+			(justify left bottom)
+		)
+	)
+	(label "{SD}"
+		(at 123.19 81.28 270)
+		(effects
+			(font
+				(size 1.27 1.27)
+			)
+			(justify right bottom)
+		)
+	)
+	(label "SD_D0"
+		(at 127 99.06 0)
+		(effects
+			(font
+				(size 1.27 1.27)
+			)
+			(justify left bottom)
 		)
 	)
 	(label "SD_CMD"
-		(at 132.08 88.9 0)
-		(effects
-			(font
-				(size 1.27 1.27)
-			)
-			(justify left bottom)
-		)
-	)
-	(label "SD_DAT2"
-		(at 132.08 83.82 0)
-		(effects
-			(font
-				(size 1.27 1.27)
-			)
-			(justify left bottom)
-		)
-	)
-	(label "SD_DAT1"
-		(at 132.08 101.6 0)
-		(effects
-			(font
-				(size 1.27 1.27)
-			)
-			(justify left bottom)
-		)
-	)
-	(label "SD_DAT3"
-		(at 132.08 86.36 0)
-		(effects
-			(font
-				(size 1.27 1.27)
-			)
-			(justify left bottom)
-		)
-	)
-	(label "{SD_DAT[0..3] SD_CMD SD_CLK}"
-		(at 129.54 81.28 90)
-		(effects
-			(font
-				(size 1.27 1.27)
-			)
-			(justify left bottom)
-		)
-	)
-	(label "SD_DAT0"
-		(at 132.08 99.06 0)
-		(effects
-			(font
-				(size 1.27 1.27)
-			)
-			(justify left bottom)
-		)
-	)
-	(label "SD_CLK"
-		(at 132.08 93.98 0)
+		(at 127 88.9 0)
+		(effects
+			(font
+				(size 1.27 1.27)
+			)
+			(justify left bottom)
+		)
+	)
+	(label "SD_D3"
+		(at 127 86.36 0)
+		(effects
+			(font
+				(size 1.27 1.27)
+			)
+			(justify left bottom)
+		)
+	)
+	(label "SD_D1"
+		(at 127 101.6 0)
 		(effects
 			(font
@@
 	(hierarchical_label "SD"
 		(shape input)
-		(at 129.54 78.74 0)
-		(effects
-			(font
-				(size 1.27 1.27)
-			)
-			(justify left)
-		)
-	)
+		(at 123.19 78.74 180)
+		(effects
+			(font
+				(size 1.27 1.27)
+			)
+			(justify right)
+		)
+	)

Commit message: final touches
Other:
- moved on the sheet: C55, J3
